File: expander_cv_input/expander_cv_input.kicad_pcb (KiCad board)
At the start: 2 copper layers, 61.8 x 128.5 mm, 14 parts

Commit message: updated files
Other:
- board text added: "JLCPCBJLCPCBJLCPCB"
- board text added: "tyrellcorp"
Changed lines of the file:
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@@
     (effects (font (size 1 1) (thickness 0.15)) (justify left bottom mirror))
+  )
+  (gr_text "JLCPCBJLCPCBJLCPCB" (at 170.3324 151.8158) (layer "B.SilkS")
+    (effects (font (size 1 1) (thickness 0.25) bold) (justify left bottom mirror))
   )
   (gr_text "stripe" (at 127.9906 92.329) (layer "B.SilkS" knockout)
     (effects (font (size 1 1) (thickness 0.15)) (justify left bottom mirror))
+  )
+  (gr_text "JLCPCBJLCPCBJLCPCB" (at 137.2616 147.5486) (layer "B.SilkS")
+    (effects (font (size 1 1) (thickness 0.25) bold) (justify left bottom mirror))
   )
   (gr_text "D" (at 170.1432 108.280716) (layer "F.SilkS")
@@
     (effects (font (size 3 2) (thickness 0.15)) (justify left bottom))
   )
-  (gr_text "CV Inputs" (at 160.7058 34.8996) (layer "F.SilkS")
+  (gr_text "CV Inputs" (at 155.2956 43.3578) (layer "F.SilkS" knockout)
     (effects (font (size 2 2) (thickness 0.15)) (justify left bottom))
   )
@@
     (effects (font (size 3 2) (thickness 0.15)) (justify left bottom))
   )
+  (gr_text "tyrellcorp" (at 164.2618 34.4932) (layer "F.SilkS")
+    (effects (font (size 1.5 1.5) (thickness 0.3) bold italic) (justify left bottom))
+  )
   (gr_text "A" (at 170.18 53.4162) (layer "F.SilkS")
