File: expander_gate_output/expander_gate_output.kicad_pcb (KiCad board)
At the start: 2 copper layers, 140 x 128.5 mm, 116 parts, among them J1 Output_A_Connector_Backboard, J16 ADDR0, J17 ADDR1, J18 ADDR2, J2 Output_B_Connector_Backboard, J3 Output_A_Connector_Frontboard, J4 Output_B_Connector_Frontboard, J5 Eurorack power, J6 CS_SELECT, J7 5V selector, U1 TXS0108EPW, U2 TXS0108EPW, U3 MCP23S17_SS

Commit message: updated files
Other:
- board text added: "JLCPCBJLCPCBJLCPCB"
- board text added: "gates"
- board text added: "tyrellcorp"
Changed lines of the file:
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@@
         (effects (font (size 1 1) (thickness 0.15)))
     )
-    (fp_text value "MCP23S17_SS" (at 0 6.25 90) (layer "F.Fab")
+    (fp_text value "MCP23S17_SS" (at 0 6.25 90) (layer "F.SilkS")
         (effects (font (size 1 1) (thickness 0.15)))
     )
@@
         (effects (font (size 1 1) (thickness 0.15)))
     )
-    (fp_text value "TXS0108EPW" (at 0.032 4.2127) (layer "F.SilkS")
+    (fp_text value "TXS0108EPW" (at 2.6736 4.6191 90) (layer "F.SilkS")
         (effects (font (size 1 1) (thickness 0.15)))
     )
@@
         (effects (font (size 1 1) (thickness 0.15)))
     )
-    (fp_text value "TXS0108EPW" (at 5.419 1.4595) (layer "F.Fab")
+    (fp_text value "TXS0108EPW" (at 0.4406 4.7107 90) (layer "F.SilkS")
         (effects (font (size 1 1) (thickness 0.15)))
     )
@@
     (fp_line (start 5.72 5.1) (end 5.72 -22.88)
       (stroke (width 0.1) (type solid)) (layer "B.Fab"))
-    (pad "1" thru_hole roundrect (at 0 0 180) (size 1.7 1.7) (drill 1) (layers "*.Cu" "*.Mask") (roundrect_rratio 0.147059)
+    (pad "1" thru_hole roundrect (at 0 0 180) (size 1.7 1.7) (drill 1) (layers "*.Cu" "*.Mask") (roundrect_rratio 0.1470588235)
       (net 40 "unconnected-(J5-Pin_1-Pad1)") (pinfunction "Pin_1") (pintype "passive"))
     (pad "2" thru_hole circle (at 2.54 0 180) (size 1.7 1.7) (drill 1) (layers "*.Cu" "*.Mask")
@@
   (gr_rect (start 171.6278 83.6422) (end 177.8092 86.1822)
     (stroke (width 0.12) (type solid)) (fill solid) (layer "B.SilkS"))
-  (gr_rect (start 145.3388 85.725) (end 139.1574 83.185)
+  (gr_rect (start 139.1574 83.185) (end 145.3388 85.725)
     (stroke (width 0.12) (type solid)) (fill solid) (layer "B.SilkS"))
   (gr_rect (start 167.0893 54.7116) (end 173.2707 57.2516)
     (stroke (width 0.12) (type solid)) (fill solid) (layer "B.SilkS"))
+  (gr_circle (center 164.5412 92.1004) (end 164.7952 92.329)
+    (stroke (width 0.12) (type default)) (fill none) (layer "F.SilkS"))
+  (gr_circle (center 156.2608 81.8134) (end 156.5656 81.9912)
+    (stroke (width 0.12) (type default)) (fill none) (layer "F.SilkS"))
+  (gr_circle (center 164.719 105.3084) (end 164.973 105.4608)
+    (stroke (width 0.12) (type default)) (fill none) (layer "F.SilkS"))
   (gr_line (start 278.1652 148.2892) (end 237.9337 148.2892)
     (stroke (width 0.05) (type solid)) (layer "Dwgs.User"))
@@
     (effects (font (size 1 1) (thickness 0.15)) (justify mirror))
   )
+  (gr_text "JLCPCBJLCPCBJLCPCB" (at 216.3064 132.842) (layer "B.SilkS")
+    (effects (font (size 1 1) (thickness 0.25) bold italic) (justify left bottom mirror))
+  )
   (gr_text "stripe" (at 166.6829 56.3626) (layer "B.SilkS" knockout)
     (effects (font (size 1 1) (thickness 0.15)) (justify left bottom mirror))
   )
+  (gr_text "JLCPCBJLCPCBJLCPCB" (at 177.7746 112.4712 90) (layer "B.SilkS")
+    (effects (font (size 1 1) (thickness 0.25) bold italic) (justify left bottom mirror))
+  )
   (gr_text "1" (at 138.6332 111.76) (layer "B.SilkS")
     (effects (font (size 1 1) (thickness 0.15)) (justify mirror))
@@
     (effects (font (size 1 1) (thickness 0.15)) (justify mirror))
   )
+  (gr_text "JLCPCBJLCPCBJLCPCB" (at 266.065 158.4452) (layer "B.SilkS")
+    (effects (font (size 1 1) (thickness 0.25) bold italic) (justify left bottom mirror))
+  )
   (gr_text "TOP" (at 192.9638 45.339) (layer "B.SilkS")
     (effects (font (size 1.5 1.5) (thickness 0.3) bold) (justify left bottom mirror))
@@
     (effects (font (size 1.5 1.5) (thickness 0.3) bold) (justify left bottom))
   )
+  (gr_text "gates" (at 254.635 42.6466) (layer "F.SilkS" knockout)
+    (effects (font (size 1.5 1.5) (thickness 0.3) bold) (justify left bottom))
+  )
   (gr_text "6" (at 254.5588 112.339965) (layer "F.SilkS")
     (effects (font (size 1.5 1.5) (thickness 0.3) bold) (justify left bottom))
@@
     (effects (font (size 1.5 1.5) (thickness 0.3) bold) (justify left bottom))
   )
+  (gr_text "tyrellcorp" (at 252.8316 34.5948) (layer "F.SilkS")
+    (effects (font (size 1.5 1.5) (thickness 0.3) bold italic) (justify left bottom))
+  )
   (gr_text "TOP" (at 173.355 45.593) (layer "F.SilkS")
