File: expander_gate_output/expander_gate_output.kicad_pcb (KiCad board)
At the start: 2 copper layers, 140 x 128.5 mm, 116 parts, among them J1 Output_A_Connector_Backboard, J16 ADDR0, J17 ADDR1, J18 ADDR2, J2 Output_B_Connector_Backboard, J3 Output_A_Connector_Frontboard, J4 Output_B_Connector_Frontboard, J5 Eurorack power, J6 CS_SELECT, J7 5V selector, U1 TXS0108EPW, U2 TXS0108EPW, U3 MCP23S17_SS

Commit message: swap accidentally flipped resistors on outputs 13+14
Parts:
- moved R27 2.72 mm to (211.3, 112.4)
- moved R28 2.64 mm to (211.3, 109.7)
- moved R26 2.54 mm to (211.5, 97.9)
- moved R25 2.52 mm to (211.5, 100.5)
Routing:
- net Net-(JACK14-Pad3): track 5.17 -> 9.13 mm
- net INT_2: track 36.3 -> 40.0 mm
- net Net-(D46-A): track 9.07 -> 5.69 mm
- net INT_1: track 36.6 -> 39.5 mm
- net Net-(D45-A): track 7.97 -> 5.91 mm
- net Net-(JACK13-Pad3): track 3.50 -> 4.91 mm
- net output_9_backboard: track 36.0 -> 37.2 mm
- net output_12_frontboard: track 72.1 -> 71.1 mm
- net +3V3: track 95.7 -> 96.4 mm
