File: expander_gate_output/Port A.kicad_sch (KiCad schematic)
At the start: 51 parts, among them J1 fuzzySI_thonkiconn

Commit message: before changing midi footprints
Parts:
- D1, D10, D11, D12, D2, D23, D24, D25, D26, D3, D4, D5, D6, D7, D8, D9: footprint Diode_SMD:D_0805_2012Metric_Pad1.15x1.40mm_HandSolder -> Diode_SMD:D_SOD-123
- R1, R2: footprint Resistor_SMD:R_0805_2012Metric_Pad1.20x1.40mm_HandSolder -> Resistor_SMD:R_0805_2012Metric
Changed lines of the file:
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@@
       (effects (font (size 1.27 1.27)))
     )
-    (property "Footprint" "Resistor_SMD:R_0805_2012Metric_Pad1.20x1.40mm_HandSolder" (at 164.8968 28.3972 90)
+    (property "Footprint" "Resistor_SMD:R_0805_2012Metric" (at 164.8968 28.3972 90)
       (effects (font (size 1.27 1.27)) hide)
     )
@@
       (effects (font (size 1.27 1.27)) (justify left))
     )
-    (property "Footprint" "Diode_SMD:D_0805_2012Metric_Pad1.15x1.40mm_HandSolder" (at 90.6018 114.808 0)
+    (property "Footprint" "Diode_SMD:D_SOD-123" (at 90.6018 114.808 0)
       (effects (font (size 1.27 1.27)) hide)
     )
@@
       (effects (font (size 1.27 1.27)) (justify left))
     )
-    (property "Footprint" "Diode_SMD:D_0805_2012Metric_Pad1.15x1.40mm_HandSolder" (at 59.2836 153.4922 0)
+    (property "Footprint" "Diode_SMD:D_SOD-123" (at 59.2836 153.4922 0)
       (effects (font (size 1.27 1.27)) hide)
     )
@@
       (effects (font (size 1.27 1.27)))
     )
-    (property "Footprint" "Resistor_SMD:R_0805_2012Metric_Pad1.20x1.40mm_HandSolder" (at 238.9632 20.2184 90)
+    (property "Footprint" "Resistor_SMD:R_0805_2012Metric" (at 238.9632 20.2184 90)
       (effects (font (size 1.27 1.27)) hide)
     )
@@
       (effects (font (size 1.27 1.27)) (justify left))
     )
-    (property "Footprint" "Diode_SMD:D_0805_2012Metric_Pad1.15x1.40mm_HandSolder" (at 90.1954 78.4352 0)
+    (property "Footprint" "Diode_SMD:D_SOD-123" (at 90.1954 78.4352 0)
       (effects (font (size 1.27 1.27)) hide)
     )
@@
       (effects (font (size 1.27 1.27)))
     )
-    (property "Footprint" "Resistor_SMD:R_0805_2012Metric_Pad1.20x1.40mm_HandSolder" (at 164.2364 74.93 90)
+    (property "Footprint" "Resistor_SMD:R_0805_2012Metric" (at 164.2364 74.93 90)
       (effects (font (size 1.27 1.27)) hide)
     )
@@
       (effects (font (size 1.27 1.27)) (justify left))
     )
-    (property "Footprint" "Diode_SMD:D_0805_2012Metric_Pad1.15x1.40mm_HandSolder" (at 31.3944 153.5938 0)
+    (property "Footprint" "Diode_SMD:D_SOD-123" (at 31.3944 153.5938 0)
       (effects (font (size 1.27 1.27)) hide)
     )
@@
       (effects (font (size 1.27 1.27)))
     )
-    (property "Footprint" "Resistor_SMD:R_0805_2012Metric_Pad1.20x1.40mm_HandSolder" (at 164.8968 19.5072 90)
+    (property "Footprint" "Resistor_SMD:R_0805_2012Metric" (at 164.8968 19.5072 90)
       (effects (font (size 1.27 1.27)) hide)
     )
@@
       (effects (font (size 1.27 1.27)) (justify left))
     )
-    (property "Footprint" "Diode_SMD:D_0805_2012Metric_Pad1.15x1.40mm_HandSolder" (at 90.6018 107.188 0)
+    (property "Footprint" "Diode_SMD:D_SOD-123" (at 90.6018 107.188 0)
       (effects (font (size 1.27 1.27)) hide)
     )
@@
       (effects (font (size 1.27 1.27)))
     )
-    (property "Footprint" "Resistor_SMD:R_0805_2012Metric_Pad1.20x1.40mm_HandSolder" (at 164.2364 83.82 90)
+    (property "Footprint" "Resistor_SMD:R_0805_2012Metric" (at 164.2364 83.82 90)
       (effects (font (size 1.27 1.27)) hide)
     )
@@
       (effects (font (size 1.27 1.27)) (justify left))
     )
-    (property "Footprint" "Diode_SMD:D_0805_2012Metric_Pad1.15x1.40mm_HandSolder" (at 90.1446 161.7472 0)
+    (property "Footprint" "Diode_SMD:D_SOD-123" (at 90.1446 161.7472 0)
       (effects (font (size 1.27 1.27)) hide)
     )
@@
       (effects (font (size 1.27 1.27)))
     )
-    (property "Footprint" "Resistor_SMD:R_0805_2012Metric_Pad1.20x1.40mm_HandSolder" (at 164.6428 46.736 90)
+    (property "Footprint" "Resistor_SMD:R_0805_2012Metric" (at 164.6428 46.736 90)
       (effects (font (size 1.27 1.27)) hide)
     )
@@
       (effects (font (size 1.27 1.27)))
     )
-    (property "Footprint" "Resistor_SMD:R_0805_2012Metric_Pad1.20x1.40mm_HandSolder" (at 239.0648 57.2008 90)
+    (property "Footprint" "Resistor_SMD:R_0805_2012Metric" (at 239.0648 57.2008 90)
       (effects (font (size 1.27 1.27)) hide)
     )
@@
       (effects (font (size 1.27 1.27)))
     )
-    (property "Footprint" "Resistor_SMD:R_0805_2012Metric_Pad1.20x1.40mm_HandSolder" (at 164.338 139.8016 90)
+    (property "Footprint" "Resistor_SMD:R_0805_2012Metric" (at 164.338 139.8016 90)
       (effects (font (size 1.27 1.27)) hide)
     )
@@
       (effects (font (size 1.27 1.27)) (justify left))
     )
-    (property "Footprint" "Diode_SMD:D_0805_2012Metric_Pad1.15x1.40mm_HandSolder" (at 90.8558 30.734 0)
+    (property "Footprint" "Diode_SMD:D_SOD-123" (at 90.8558 30.734 0)
       (effects (font (size 1.27 1.27)) hide)
     )
@@
       (effects (font (size 1.27 1.27)))
     )
-    (property "Footprint" "Resistor_SMD:R_0805_2012Metric_Pad1.20x1.40mm_HandSolder" (at 164.338 130.9116 90)
+    (property "Footprint" "Resistor_SMD:R_0805_2012Metric" (at 164.338 130.9116 90)
       (effects (font (size 1.27 1.27)) hide)
     )
@@
       (effects (font (size 1.27 1.27)) (justify left))
     )
-    (property "Footprint" "Diode_SMD:D_0805_2012Metric_Pad1.15x1.40mm_HandSolder" (at 90.8558 23.114 0)
+    (property "Footprint" "Diode_SMD:D_SOD-123" (at 90.8558 23.114 0)
       (effects (font (size 1.27 1.27)) hide)
     )
@@
       (effects (font (size 1.27 1.27)))
     )
-    (property "Footprint" "Resistor_SMD:R_0805_2012Metric_Pad1.20x1.40mm_HandSolder" (at 164.084 160.528 90)
+    (property "Footprint" "Resistor_SMD:R_0805_2012Metric" (at 164.084 160.528 90)
       (effects (font (size 1.27 1.27)) hide)
     )
@@
       (effects (font (size 1.27 1.27)) (justify left))
     )
-    (property "Footprint" "Diode_SMD:D_0805_2012Metric_Pad1.15x1.40mm_HandSolder" (at 90.297 142.0368 0)
+    (property "Footprint" "Diode_SMD:D_SOD-123" (at 90.297 142.0368 0)
       (effects (font (size 1.27 1.27)) hide)
     )
@@
       (effects (font (size 1.27 1.27)))
     )
-    (property "Footprint" "Resistor_SMD:R_0805_2012Metric_Pad1.20x1.40mm_HandSolder" (at 164.6428 55.626 90)
+    (property "Footprint" "Resistor_SMD:R_0805_2012Metric" (at 164.6428 55.626 90)
       (effects (font (size 1.27 1.27)) hide)
     )
@@
       (effects (font (size 1.27 1.27)))
     )
-    (property "Footprint" "Resistor_SMD:R_0805_2012Metric_Pad1.20x1.40mm_HandSolder" (at 164.084 151.638 90)
+    (property "Footprint" "Resistor_SMD:R_0805_2012Metric" (at 164.084 151.638 90)
       (effects (font (size 1.27 1.27)) hide)
     )
@@
       (effects (font (size 1.27 1.27)) (justify left))
     )
-    (property "Footprint" "Diode_SMD:D_0805_2012Metric_Pad1.15x1.40mm_HandSolder" (at 39.0144 153.5938 0)
+    (property "Footprint" "Diode_SMD:D_SOD-123" (at 39.0144 153.5938 0)
       (effects (font (size 1.27 1.27)) hide)
     )
@@
       (effects (font (size 1.27 1.27)) (justify left))
     )
-    (property "Footprint" "Diode_SMD:D_0805_2012Metric_Pad1.15x1.40mm_HandSolder" (at 66.9036 153.4922 0)
+    (property "Footprint" "Diode_SMD:D_SOD-123" (at 66.9036 153.4922 0)
       (effects (font (size 1.27 1.27)) hide)
     )
@@
       (effects (font (size 1.27 1.27)))
     )
-    (property "Footprint" "Resistor_SMD:R_0805_2012Metric_Pad1.20x1.40mm_HandSolder" (at 238.9632 29.1084 90)
+    (property "Footprint" "Resistor_SMD:R_0805_2012Metric" (at 238.9632 29.1084 90)
       (effects (font (size 1.27 1.27)) hide)
     )
@@
       (effects (font (size 1.27 1.27)) (justify left))
     )
-    (property "Footprint" "Diode_SMD:D_0805_2012Metric_Pad1.15x1.40mm_HandSolder" (at 90.6018 58.2676 0)
+    (property "Footprint" "Diode_SMD:D_SOD-123" (at 90.6018 58.2676 0)
       (effects (font (size 1.27 1.27)) hide)
     )
@@
       (effects (font (size 1.27 1.27)))
     )
-    (property "Footprint" "Resistor_SMD:R_0805_2012Metric_Pad1.20x1.40mm_HandSolder" (at 164.6428 112.1664 90)
+    (property "Footprint" "Resistor_SMD:R_0805_2012Metric" (at 164.6428 112.1664 90)
       (effects (font (size 1.27 1.27)) hide)
     )
@@
       (effects (font (size 1.27 1.27)) (justify left))
     )
-    (property "Footprint" "Diode_SMD:D_0805_2012Metric_Pad1.15x1.40mm_HandSolder" (at 90.1954 86.0552 0)
+    (property "Footprint" "Diode_SMD:D_SOD-123" (at 90.1954 86.0552 0)
       (effects (font (size 1.27 1.27)) hide)
     )
@@
       (effects (font (size 1.27 1.27)) (justify left))
     )
-    (property "Footprint" "Diode_SMD:D_0805_2012Metric_Pad1.15x1.40mm_HandSolder" (at 90.6018 50.6476 0)
+    (property "Footprint" "Diode_SMD:D_SOD-123" (at 90.6018 50.6476 0)
       (effects (font (size 1.27 1.27)) hide)
     )
@@
       (effects (font (size 1.27 1.27)))
     )
-    (property "Footprint" "Resistor_SMD:R_0805_2012Metric_Pad1.20x1.40mm_HandSolder" (at 164.6428 103.2764 90)
+    (property "Footprint" "Resistor_SMD:R_0805_2012Metric" (at 164.6428 103.2764 90)
       (effects (font (size 1.27 1.27)) hide)
     )
@@
       (effects (font (size 1.27 1.27)) (justify left))
     )
-    (property "Footprint" "Diode_SMD:D_0805_2012Metric_Pad1.15x1.40mm_HandSolder" (at 90.297 134.4168 0)
+    (property "Footprint" "Diode_SMD:D_SOD-123" (at 90.297 134.4168 0)
       (effects (font (size 1.27 1.27)) hide)
     )
@@
       (effects (font (size 1.27 1.27)) (justify left))
     )
-    (property "Footprint" "Diode_SMD:D_0805_2012Metric_Pad1.15x1.40mm_HandSolder" (at 90.1446 169.3672 0)
+    (property "Footprint" "Diode_SMD:D_SOD-123" (at 90.1446 169.3672 0)
       (effects (font (size 1.27 1.27)) hide)
     )
@@
       (effects (font (size 1.27 1.27)))
     )
-    (property "Footprint" "Resistor_SMD:R_0805_2012Metric_Pad1.20x1.40mm_HandSolder" (at 239.0648 48.3108 90)
-      (effects (font (size 1.27 1.27)) hide)
-    )
+    (property "Footprint" "Resistor_SMD:R_0805_2012Metric" (at 239.0648 48.3108 90)
+      (effects (font (size 1.27 1.27)) hide)
+    )
