File: expander_gate_output/Port B.kicad_sch (KiCad schematic)
At the start: 51 parts, among them J1 fuzzySI_thonkiconn

Commit message: before changing midi footprints
Parts:
- D1, D10, D11, D12, D2, D23, D24, D25, D26, D3, D4, D5, D6, D7, D8, D9: footprint Diode_SMD:D_0805_2012Metric_Pad1.15x1.40mm_HandSolder -> Diode_SMD:D_SOD-123
- R1, R2: footprint Resistor_SMD:R_0805_2012Metric_Pad1.20x1.40mm_HandSolder -> Resistor_SMD:R_0805_2012Metric
Changed lines of the file:
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@@
       (effects (font (size 1.27 1.27)))
     )
-    (property "Footprint" "Resistor_SMD:R_0805_2012Metric_Pad1.20x1.40mm_HandSolder" (at 165.2778 164.1094 90)
+    (property "Footprint" "Resistor_SMD:R_0805_2012Metric" (at 165.2778 164.1094 90)
       (effects (font (size 1.27 1.27)) hide)
     )
@@
       (effects (font (size 1.27 1.27)) (justify left))
     )
-    (property "Footprint" "Diode_SMD:D_0805_2012Metric_Pad1.15x1.40mm_HandSolder" (at 91.3384 172.9486 0)
+    (property "Footprint" "Diode_SMD:D_SOD-123" (at 91.3384 172.9486 0)
       (effects (font (size 1.27 1.27)) hide)
     )
@@
       (effects (font (size 1.27 1.27)) (justify left))
     )
-    (property "Footprint" "Diode_SMD:D_0805_2012Metric_Pad1.15x1.40mm_HandSolder" (at 91.7956 110.7694 0)
+    (property "Footprint" "Diode_SMD:D_SOD-123" (at 91.7956 110.7694 0)
       (effects (font (size 1.27 1.27)) hide)
     )
@@
       (effects (font (size 1.27 1.27)))
     )
-    (property "Footprint" "Resistor_SMD:R_0805_2012Metric_Pad1.20x1.40mm_HandSolder" (at 240.157 32.6898 90)
+    (property "Footprint" "Resistor_SMD:R_0805_2012Metric" (at 240.157 32.6898 90)
       (effects (font (size 1.27 1.27)) hide)
     )
@@
       (effects (font (size 1.27 1.27)) (justify left))
     )
-    (property "Footprint" "Diode_SMD:D_0805_2012Metric_Pad1.15x1.40mm_HandSolder" (at 91.3384 165.3286 0)
+    (property "Footprint" "Diode_SMD:D_SOD-123" (at 91.3384 165.3286 0)
       (effects (font (size 1.27 1.27)) hide)
     )
@@
       (effects (font (size 1.27 1.27)))
     )
-    (property "Footprint" "Resistor_SMD:R_0805_2012Metric_Pad1.20x1.40mm_HandSolder" (at 165.2778 155.2194 90)
+    (property "Footprint" "Resistor_SMD:R_0805_2012Metric" (at 165.2778 155.2194 90)
       (effects (font (size 1.27 1.27)) hide)
     )
@@
       (effects (font (size 1.27 1.27)) (justify left))
     )
-    (property "Footprint" "Diode_SMD:D_0805_2012Metric_Pad1.15x1.40mm_HandSolder" (at 40.2082 157.1752 0)
+    (property "Footprint" "Diode_SMD:D_SOD-123" (at 40.2082 157.1752 0)
       (effects (font (size 1.27 1.27)) hide)
     )
@@
       (effects (font (size 1.27 1.27)))
     )
-    (property "Footprint" "Resistor_SMD:R_0805_2012Metric_Pad1.20x1.40mm_HandSolder" (at 240.157 23.7998 90)
+    (property "Footprint" "Resistor_SMD:R_0805_2012Metric" (at 240.157 23.7998 90)
       (effects (font (size 1.27 1.27)) hide)
     )
@@
       (effects (font (size 1.27 1.27)))
     )
-    (property "Footprint" "Resistor_SMD:R_0805_2012Metric_Pad1.20x1.40mm_HandSolder" (at 165.8874 106.8578 90)
+    (property "Footprint" "Resistor_SMD:R_0805_2012Metric" (at 165.8874 106.8578 90)
       (effects (font (size 1.27 1.27)) hide)
     )
@@
       (effects (font (size 1.27 1.27)) (justify left))
     )
-    (property "Footprint" "Diode_SMD:D_0805_2012Metric_Pad1.15x1.40mm_HandSolder" (at 91.3892 89.6366 0)
+    (property "Footprint" "Diode_SMD:D_SOD-123" (at 91.3892 89.6366 0)
       (effects (font (size 1.27 1.27)) hide)
     )
@@
       (effects (font (size 1.27 1.27)) (justify left))
     )
-    (property "Footprint" "Diode_SMD:D_0805_2012Metric_Pad1.15x1.40mm_HandSolder" (at 91.3892 82.0166 0)
+    (property "Footprint" "Diode_SMD:D_SOD-123" (at 91.3892 82.0166 0)
       (effects (font (size 1.27 1.27)) hide)
     )
@@
       (effects (font (size 1.27 1.27)))
     )
-    (property "Footprint" "Resistor_SMD:R_0805_2012Metric_Pad1.20x1.40mm_HandSolder" (at 240.2586 60.7822 90)
+    (property "Footprint" "Resistor_SMD:R_0805_2012Metric" (at 240.2586 60.7822 90)
       (effects (font (size 1.27 1.27)) hide)
     )
@@
       (effects (font (size 1.27 1.27)) (justify left))
     )
-    (property "Footprint" "Diode_SMD:D_0805_2012Metric_Pad1.15x1.40mm_HandSolder" (at 32.5882 157.1752 0)
+    (property "Footprint" "Diode_SMD:D_SOD-123" (at 32.5882 157.1752 0)
       (effects (font (size 1.27 1.27)) hide)
     )
@@
       (effects (font (size 1.27 1.27)))
     )
-    (property "Footprint" "Resistor_SMD:R_0805_2012Metric_Pad1.20x1.40mm_HandSolder" (at 166.0906 23.0886 90)
+    (property "Footprint" "Resistor_SMD:R_0805_2012Metric" (at 166.0906 23.0886 90)
       (effects (font (size 1.27 1.27)) hide)
     )
@@
       (effects (font (size 1.27 1.27)))
     )
-    (property "Footprint" "Resistor_SMD:R_0805_2012Metric_Pad1.20x1.40mm_HandSolder" (at 165.4302 78.5114 90)
+    (property "Footprint" "Resistor_SMD:R_0805_2012Metric" (at 165.4302 78.5114 90)
       (effects (font (size 1.27 1.27)) hide)
     )
@@
       (effects (font (size 1.27 1.27)))
     )
-    (property "Footprint" "Resistor_SMD:R_0805_2012Metric_Pad1.20x1.40mm_HandSolder" (at 165.4302 87.4014 90)
+    (property "Footprint" "Resistor_SMD:R_0805_2012Metric" (at 165.4302 87.4014 90)
       (effects (font (size 1.27 1.27)) hide)
     )
@@
       (effects (font (size 1.27 1.27)))
     )
-    (property "Footprint" "Resistor_SMD:R_0805_2012Metric_Pad1.20x1.40mm_HandSolder" (at 165.8366 59.2074 90)
+    (property "Footprint" "Resistor_SMD:R_0805_2012Metric" (at 165.8366 59.2074 90)
       (effects (font (size 1.27 1.27)) hide)
     )
@@
       (effects (font (size 1.27 1.27)))
     )
-    (property "Footprint" "Resistor_SMD:R_0805_2012Metric_Pad1.20x1.40mm_HandSolder" (at 165.5826 143.383 90)
+    (property "Footprint" "Resistor_SMD:R_0805_2012Metric" (at 165.5826 143.383 90)
       (effects (font (size 1.27 1.27)) hide)
     )
@@
       (effects (font (size 1.27 1.27)) (justify left))
     )
-    (property "Footprint" "Diode_SMD:D_0805_2012Metric_Pad1.15x1.40mm_HandSolder" (at 68.0974 157.0736 0)
+    (property "Footprint" "Diode_SMD:D_SOD-123" (at 68.0974 157.0736 0)
       (effects (font (size 1.27 1.27)) hide)
     )
@@
       (effects (font (size 1.27 1.27)))
     )
-    (property "Footprint" "Resistor_SMD:R_0805_2012Metric_Pad1.20x1.40mm_HandSolder" (at 240.2586 51.8922 90)
+    (property "Footprint" "Resistor_SMD:R_0805_2012Metric" (at 240.2586 51.8922 90)
       (effects (font (size 1.27 1.27)) hide)
     )
@@
       (effects (font (size 1.27 1.27)) (justify left))
     )
-    (property "Footprint" "Diode_SMD:D_0805_2012Metric_Pad1.15x1.40mm_HandSolder" (at 91.7956 61.849 0)
+    (property "Footprint" "Diode_SMD:D_SOD-123" (at 91.7956 61.849 0)
       (effects (font (size 1.27 1.27)) hide)
     )
@@
       (effects (font (size 1.27 1.27)) (justify left))
     )
-    (property "Footprint" "Diode_SMD:D_0805_2012Metric_Pad1.15x1.40mm_HandSolder" (at 91.4908 145.6182 0)
+    (property "Footprint" "Diode_SMD:D_SOD-123" (at 91.4908 145.6182 0)
       (effects (font (size 1.27 1.27)) hide)
     )
@@
       (effects (font (size 1.27 1.27)) (justify left))
     )
-    (property "Footprint" "Diode_SMD:D_0805_2012Metric_Pad1.15x1.40mm_HandSolder" (at 91.4908 137.9982 0)
+    (property "Footprint" "Diode_SMD:D_SOD-123" (at 91.4908 137.9982 0)
       (effects (font (size 1.27 1.27)) hide)
     )
@@
       (effects (font (size 1.27 1.27)) (justify left))
     )
-    (property "Footprint" "Diode_SMD:D_0805_2012Metric_Pad1.15x1.40mm_HandSolder" (at 60.4774 157.0736 0)
+    (property "Footprint" "Diode_SMD:D_SOD-123" (at 60.4774 157.0736 0)
       (effects (font (size 1.27 1.27)) hide)
     )
@@
       (effects (font (size 1.27 1.27)) (justify left))
     )
-    (property "Footprint" "Diode_SMD:D_0805_2012Metric_Pad1.15x1.40mm_HandSolder" (at 91.7956 54.229 0)
+    (property "Footprint" "Diode_SMD:D_SOD-123" (at 91.7956 54.229 0)
       (effects (font (size 1.27 1.27)) hide)
     )
@@
       (effects (font (size 1.27 1.27)) (justify left))
     )
-    (property "Footprint" "Diode_SMD:D_0805_2012Metric_Pad1.15x1.40mm_HandSolder" (at 92.0496 34.3154 0)
+    (property "Footprint" "Diode_SMD:D_SOD-123" (at 92.0496 34.3154 0)
       (effects (font (size 1.27 1.27)) hide)
     )
@@
       (effects (font (size 1.27 1.27)))
     )
-    (property "Footprint" "Resistor_SMD:R_0805_2012Metric_Pad1.20x1.40mm_HandSolder" (at 165.8874 115.7478 90)
+    (property "Footprint" "Resistor_SMD:R_0805_2012Metric" (at 165.8874 115.7478 90)
       (effects (font (size 1.27 1.27)) hide)
     )
@@
       (effects (font (size 1.27 1.27)))
     )
-    (property "Footprint" "Resistor_SMD:R_0805_2012Metric_Pad1.20x1.40mm_HandSolder" (at 165.8366 50.3174 90)
+    (property "Footprint" "Resistor_SMD:R_0805_2012Metric" (at 165.8366 50.3174 90)
       (effects (font (size 1.27 1.27)) hide)
     )
@@
       (effects (font (size 1.27 1.27)))
     )
-    (property "Footprint" "Resistor_SMD:R_0805_2012Metric_Pad1.20x1.40mm_HandSolder" (at 166.0906 31.9786 90)
+    (property "Footprint" "Resistor_SMD:R_0805_2012Metric" (at 166.0906 31.9786 90)
       (effects (font (size 1.27 1.27)) hide)
     )
@@
       (effects (font (size 1.27 1.27)) (justify left))
     )
-    (property "Footprint" "Diode_SMD:D_0805_2012Metric_Pad1.15x1.40mm_HandSolder" (at 91.7956 118.3894 0)
+    (property "Footprint" "Diode_SMD:D_SOD-123" (at 91.7956 118.3894 0)
       (effects (font (size 1.27 1.27)) hide)
     )
@@
       (effects (font (size 1.27 1.27)) (justify left))
     )
-    (property "Footprint" "Diode_SMD:D_0805_2012Metric_Pad1.15x1.40mm_HandSolder" (at 92.0496 26.6954 0)
+    (property "Footprint" "Diode_SMD:D_SOD-123" (at 92.0496 26.6954 0)
       (effects (font (size 1.27 1.27)) hide)
     )
@@
       (effects (font (size 1.27 1.27)))
     )
-    (property "Footprint" "Resistor_SMD:R_0805_2012Metric_Pad1.20x1.40mm_HandSolder" (at 165.5826 134.493 90)
+    (property "Footprint" "Resistor_SMD:R_0805_2012Metric" (at 165.5826 134.493 90)
       (effects (font (size 1.27 1.27)) hide)
     )
