File: expander_gate_output/expander_gate_output - Copy.kicad_pcb (KiCad board)
At the start: 2 copper layers, 140 x 128.5 mm, 116 parts, among them J1 Output_A_Connector_Backboard, J16 ADDR0, J17 ADDR1, J18 ADDR2, J2 Output_B_Connector_Backboard, J3 Output_A_Connector_Frontboard, J4 Output_B_Connector_Frontboard, J5 Eurorack power, J6 CS_SELECT, J7 5V selector, U1 TXS0108EPW, U2 TXS0108EPW, U3 MCP23S17_SS

Commit message: before changing midi footprints
Parts:
- removed EXPANDER_THRU, GATE_SPI_OUTPUT_EXPANDER1: 16 pin header, Connector_PinHeader_2.54mm:PinHeader_2x08_P2.54mm_Vertical
- added SPI Expander THRU: NOT POWER!!, Connector_PinHeader_2.54mm:PinHeader_2x08_P2.54mm_Vertical, B.Cu at (176.2, 85.1)
- added SPI Expander to Host: 16 pin header, Connector_PinHeader_2.54mm:PinHeader_2x08_P2.54mm_Vertical, B.Cu at (143.3, 84.6)
- D1, D10, D11, D12, D13, D14, D15, D16, D2, D25, D26, D27, D28, D29, D3, D30, D31, D32, D33, D34, D35, D36, D37, D38, D39, D4, D40, D5, D6, D7, D8, D9: footprint Diode_SMD:D_SOD-123 -> Diode_SMD:D_0805_2012Metric
- moved D36 17.5 mm to (161.8, 133.0), turned to 180 degrees
- moved D16 16.8 mm to (164.0, 65.3)
- moved D37 16.3 mm to (157.6, 135.9)
- moved D38 15.9 mm to (156.1, 138.1)
- moved D9 13.3 mm to (154.2, 53.2), turned to 0 degrees
- moved D5 12.9 mm to (156.8, 50.6), turned to 0 degrees
- moved D1 12.4 mm to (160.6, 48.3)
- moved D4 9.71 mm to (158.1, 70.3)
- moved D15 8.92 mm to (166.0, 48.3)
- moved D8 8.77 mm to (152.7, 67.9), turned to 0 degrees
- moved D29 8.56 mm to (149.7, 138.1), turned to 0 degrees
- moved D35 8.29 mm to (162.8, 126.6)
- moved D40 8.10 mm to (165.4, 134.9)
- moved D6 7.79 mm to (159.8, 67.2)
- moved D39 7.63 mm to (165.4, 138.2)
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Routing:
- net +5V: track 212.6 -> 182.8 mm, vias 15 -> 12
- net GND: track 198.2 -> 206.1 mm, vias 13 -> 15
- net +5V from main: track 36.3 -> 39.0 mm, vias 0 -> 1
- net output_16_backboard: track 40.1 -> 41.9 mm, vias 1 -> 2
- net output_1_backboard: track 35.9 -> 37.3 mm, vias 2 -> 0
- net output_10_backboard: track 37.0 -> 35.7 mm
- net output_4_backboard: track 33.7 -> 32.7 mm
- net MOSI: track 50.9 -> 49.9 mm
- net output_14_backboard: track 38.5 -> 39.4 mm
- net output_7_backboard: track 32.3 -> 31.6 mm
- net Net-(D18-A): track 6.21 -> 5.58 mm
- net output_3_backboard: track 34.5 -> 34.0 mm
Other:
- board text added: "gates"
- board text removed: "I shoot arrows of time in all directions"
- board text removed: "Tannhäuser gates"
