File: expander_midi/expander_midi.kicad_pcb (KiCad board)
At the start: 2 copper layers, 90.3 x 128.5 mm, 73 parts

Commit message: rough layout of single midi expander
Parts:
- removed C7, C8: 100n, Capacitor_SMD:C_0805_2012Metric
- removed JMIDIIN5, JMIDIIN6, JMIDIIN7, JMIDIIN8, JMIDIOUT5, JMIDIOUT6, JMIDIOUT7, JMIDIOUT8: MIDI In Jack 3.5mm stereo jack, doctea:Jack_3.5mm_QingPu_WQP-PJ398SM_TRS_Vertical_CircularHoles
- removed MIDI_EXPANDER_MAIN1: 20 pin header, Connector_PinHeader_2.54mm:PinHeader_2x10_P2.54mm_Vertical
- removed R21, R22: 220R, Resistor_SMD:R_0805_2012Metric
- removed R23, R24: 470R, Resistor_SMD:R_0805_2012Metric
- removed R25, R26, R27, R28, R29, R30, R31, R32, R33, R34, R35, R36, R37, R38, R39, R40: 47R, Resistor_SMD:R_0805_2012Metric
- removed ULPZWmidi5, ULPZWmidi6, ULPZWmidi7, ULPZWmidi8: HCPL-0631, Package_SO:SOIC-8_3.9x4.9mm_P1.27mm
- added MIDI_EXPANDER_1: Conn_02x05_Counter_Clockwise, Connector_PinHeader_2.54mm:PinHeader_2x05_P2.54mm_Vertical, B.Cu at (204.5, 134.5)
- added REF**: PinHeader_2x06_P2.54mm_Vertical, Connector_PinHeader_2.54mm:PinHeader_2x06_P2.54mm_Vertical, F.Cu at (204.0, 55.2)
- added REF**: PinHeader_1x06_P2.54mm_Vertical, Connector_PinHeader_2.54mm:PinHeader_1x06_P2.54mm_Vertical, F.Cu at (204.0, 158.4)
- added REF**: PinSocket_2x06_P2.54mm_Vertical, Connector_PinSocket_2.54mm:PinSocket_2x06_P2.54mm_Vertical, B.Cu at (178.8, 55.2)
- added REF**: PinHeader_1x06_P2.54mm_Vertical, Connector_PinHeader_2.54mm:PinHeader_1x06_P2.54mm_Vertical, B.Cu at (177.6, 158.6)
- added U1: LD1117, Package_TO_SOT_SMD:SOT-223-3_TabPin2, F.Cu at (205.2, 147.0)
- C1, C2: value 100n -> 100nF; footprint Capacitor_SMD:C_0805_2012Metric -> Capacitor_THT:C_Axial_L5.1mm_D3.1mm_P7.50mm_Horizontal
- C3, C4, C5: footprint Capacitor_SMD:C_0805_2012Metric -> Capacitor_THT:C_Axial_L5.1mm_D3.1mm_P7.50mm_Horizontal
- C6: footprint Capacitor_SMD:C_0805_2012Metric -> Capacitor_THT:C_Axial_L5.1mm_D3.1mm_P7.50mm_Horizontal; moved to F.Cu
- R1, R4: value 220R -> 47R; footprint Resistor_SMD:R_0805_2012Metric -> Resistor_THT:R_Axial_DIN0207_L6.3mm_D2.5mm_P7.62mm_Horizontal
- R10, R15, R16: footprint Resistor_SMD:R_0805_2012Metric -> Resistor_THT:R_Axial_DIN0207_L6.3mm_D2.5mm_P7.62mm_Horizontal; moved to F.Cu
- R11: footprint Resistor_SMD:R_0805_2012Metric -> Resistor_THT:R_Axial_DIN0207_L6.3mm_D2.5mm_P7.62mm_Horizontal
- R12, R17: value 470R -> 220R; footprint Resistor_SMD:R_0805_2012Metric -> Resistor_THT:R_Axial_DIN0207_L6.3mm_D2.5mm_P7.62mm_Horizontal; moved to F.Cu
- R13, R14, R19, R20: value 220R -> 470R; footprint Resistor_SMD:R_0805_2012Metric -> Resistor_THT:R_Axial_DIN0207_L6.3mm_D2.5mm_P7.62mm_Horizontal; moved to F.Cu
- R18, R9: value 470R -> 220R; footprint Resistor_SMD:R_0805_2012Metric -> Resistor_THT:R_Axial_DIN0207_L6.3mm_D2.5mm_P7.62mm_Horizontal
- R2, R5, R7, R8: value 220R -> 47R; footprint Resistor_SMD:R_0805_2012Metric -> Resistor_THT:R_Axial_DIN0207_L6.3mm_D2.5mm_P7.62mm_Horizontal; moved to F.Cu
- R3: value 470R -> 47R; footprint Resistor_SMD:R_0805_2012Metric -> Resistor_THT:R_Axial_DIN0207_L6.3mm_D2.5mm_P7.62mm_Horizontal; moved to F.Cu
- R6: value 470R -> 47R; footprint Resistor_SMD:R_0805_2012Metric -> Resistor_THT:R_Axial_DIN0207_L6.3mm_D2.5mm_P7.62mm_Horizontal
- ULPZWmidi1, ULPZWmidi2, ULPZWmidi3, ULPZWmidi4: moved to F.Cu
- moved R2 88.7 mm to (175.8, 155.4), turned to 90 degrees
- moved R3 86.6 mm to (175.9, 142.9), turned to 90 degrees
- moved R6 63.7 mm to (179.2, 132.9), turned to 0 degrees
- moved JMIDIOUT2 55.8 mm to (190.5, 151.6)
- moved JMIDIOUT3 55.8 mm to (190.5, 139.1)
- moved JMIDIOUT4 55.8 mm to (190.5, 126.5)
- moved JMIDIOUT1 55.8 mm to (190.5, 114.0)
- moved R7 52.4 mm to (187.0, 145.4)
- moved R13 49.7 mm to (215.6, 73.2), turned to 90 degrees
- moved R19 49.5 mm to (215.5, 98.5), turned to 90 degrees
- moved R16 42.6 mm to (203.5, 90.7), turned to -90 degrees
- moved R10 41.8 mm to (204.3, 65.4), turned to -90 degrees
- moved R5 40.8 mm to (175.7, 117.8), turned to 90 degrees
- moved R1 40.7 mm to (186.7, 107.7)
- moved R8 40.5 mm to (175.9, 130.4), turned to 90 degrees
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Connections:
- C2 pad 1: +5V -> +3V3
- JMIDIIN1 pad R: Net-(ULPZWmidi1-C2) -> MIDI_IN_R_1
- JMIDIIN1 pad T: Net-(ULPZWmidi1-C1) -> MIDI_IN_T_1
- JMIDIIN2 pad R: Net-(ULPZWmidi2-C2) -> MIDI_IN_R_3
- JMIDIIN2 pad T: Net-(ULPZWmidi2-C1) -> MIDI_IN_T_3
- JMIDIIN3 pad R: Net-(ULPZWmidi3-C2) -> MIDI_IN_R_4
- JMIDIIN3 pad T: Net-(ULPZWmidi3-C1) -> MIDI_IN_T_4
- JMIDIIN4 pad R: Net-(ULPZWmidi4-C2) -> MIDI_IN_R_2
- JMIDIIN4 pad T: Net-(ULPZWmidi4-C1) -> MIDI_IN_T_2
- R1 pad 1: Net-(ULPZWmidi1-A1) -> Net-(JMIDIOUT1-PadR)
- R1 pad 2: Net-(ULPZWmidi1-C2) -> +3V3
- R10 pad 1: Net-(ULPZWmidi4-A1) -> Net-(ULPZWmidi1-A2)
- R10 pad 2: Net-(ULPZWmidi4-C2) -> MIDI_IN_T_1
- R11 pad 1: Net-(ULPZWmidi4-A2) -> Net-(ULPZWmidi2-A1)
- R11 pad 2: Net-(ULPZWmidi4-C1) -> MIDI_IN_R_3
- R12 pad 1: +3V3 -> Net-(ULPZWmidi2-A2)
- R12 pad 2: MIDI_4_RX -> MIDI_IN_T_3
- R13 pad 1: Net-(ULPZWmidi5-A1) -> +3V3
- R13 pad 2: Net-(ULPZWmidi5-C2) -> MIDI_1_RX
- R14 pad 1: Net-(ULPZWmidi5-A2) -> +3V3
- R14 pad 2: Net-(ULPZWmidi5-C1) -> MIDI_3_RX
- R15 pad 1: Net-(ULPZWmidi6-A1) -> Net-(ULPZWmidi3-A1)
- R15 pad 2: Net-(ULPZWmidi6-C2) -> MIDI_IN_R_4
- R16 pad 1: Net-(ULPZWmidi6-A2) -> Net-(ULPZWmidi3-A2)
- R16 pad 2: Net-(ULPZWmidi6-C1) -> MIDI_IN_T_4
- R17 pad 1: +3V3 -> Net-(ULPZWmidi4-A1)
- R17 pad 2: MIDI_5_RX -> MIDI_IN_R_2
- R18 pad 1: +3V3 -> Net-(ULPZWmidi4-A2)
- R18 pad 2: MIDI_7_RX -> MIDI_IN_T_2
- R19 pad 1: Net-(ULPZWmidi7-A1) -> +3V3
- R19 pad 2: Net-(ULPZWmidi7-C2) -> MIDI_4_RX
- R2 pad 1: Net-(ULPZWmidi1-A2) -> Net-(JMIDIOUT2-PadR)
- R2 pad 2: Net-(ULPZWmidi1-C1) -> +3V3
- R20 pad 1: Net-(ULPZWmidi7-A2) -> +3V3
- R20 pad 2: Net-(ULPZWmidi7-C1) -> MIDI_2_RX
- R3 pad 1: +3V3 -> Net-(JMIDIOUT3-PadR)
- R3 pad 2: MIDI_1_RX -> +3V3
- R4 pad 1: Net-(ULPZWmidi2-A1) -> Net-(JMIDIOUT4-PadR)
- R4 pad 2: Net-(ULPZWmidi2-C2) -> +3V3
- R5 pad 1: Net-(ULPZWmidi2-A2) -> Net-(JMIDIOUT1-PadT)
- R5 pad 2: Net-(ULPZWmidi2-C1) -> MIDI_1_TX
- R6 pad 1: +3V3 -> Net-(JMIDIOUT2-PadT)
- R6 pad 2: MIDI_2_RX -> MIDI_2_TX
- R7 pad 1: Net-(ULPZWmidi3-A1) -> Net-(JMIDIOUT3-PadT)
- R7 pad 2: Net-(ULPZWmidi3-C2) -> MIDI_3_TX
- R8 pad 1: Net-(ULPZWmidi3-A2) -> Net-(JMIDIOUT4-PadT)
- R8 pad 2: Net-(ULPZWmidi3-C1) -> MIDI_4_TX
- R9 pad 1: +3V3 -> Net-(ULPZWmidi1-A1)
- R9 pad 2: MIDI_3_RX -> MIDI_IN_R_1
- ULPZWmidi1 pad 2: Net-(ULPZWmidi1-C1) -> MIDI_IN_T_1
- ULPZWmidi1 pad 3: Net-(ULPZWmidi1-C2) -> MIDI_IN_R_1
- ULPZWmidi2 pad 2: Net-(ULPZWmidi2-C1) -> MIDI_IN_T_3
- ULPZWmidi2 pad 3: Net-(ULPZWmidi2-C2) -> MIDI_IN_R_3
- ULPZWmidi2 pad 6: MIDI_2_RX -> MIDI_3_RX
- ULPZWmidi2 pad 7: MIDI_2_RX -> MIDI_3_RX
- ULPZWmidi3 pad 2: Net-(ULPZWmidi3-C1) -> MIDI_IN_T_4
- ULPZWmidi3 pad 3: Net-(ULPZWmidi3-C2) -> MIDI_IN_R_4
- ULPZWmidi3 pad 6: MIDI_3_RX -> MIDI_4_RX
- ULPZWmidi3 pad 7: MIDI_3_RX -> MIDI_4_RX
- ULPZWmidi4 pad 2: Net-(ULPZWmidi4-C1) -> MIDI_IN_T_2
- ULPZWmidi4 pad 3: Net-(ULPZWmidi4-C2) -> MIDI_IN_R_2
- ULPZWmidi4 pad 6: MIDI_4_RX -> MIDI_2_RX
- ULPZWmidi4 pad 7: MIDI_4_RX -> MIDI_2_RX
Routing:
- net MIDI_IN_T_2: track 0.00 -> 132.4 mm
- net MIDI_IN_R_2: track 0.00 -> 123.7 mm
- net MIDI_6_RX: track 121.4 -> 0.00 mm, vias 2 -> 0
- net MIDI_8_RX: track 119.6 -> 0.00 mm, vias 1 -> 0
- net MIDI_5_RX: track 106.0 -> 0.00 mm, vias 1 -> 0
- net MIDI_IN_T_4: track 0.00 -> 104.2 mm
- net MIDI_6_TX: track 95.5 -> 0.00 mm, vias 2 -> 0
- net MIDI_IN_R_4: track 0.00 -> 93.7 mm, vias 0 -> 1
- net MIDI_7_RX: track 88.1 -> 0.00 mm, vias 2 -> 0
- net MIDI_IN_T_3: track 0.00 -> 79.4 mm
- net MIDI_8_TX: track 60.6 -> 0.00 mm
- net MIDI_IN_R_3: track 0.00 -> 59.6 mm
- net MIDI_1_RX: track 27.7 -> 84.5 mm, vias 1 -> 2
- net MIDI_1_TX: track 23.5 -> 77.4 mm
- net +3V3: track 208.2 -> 156.4 mm, vias 2 -> 1
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- added copper zone on B.Cu, net +3V3
- added copper zone on F.Cu, net +5V
Other:
- board size 90.3 x 128.5 mm -> 70.4 x 128.5 mm
- board text removed: "5"
- board text removed: "6"
- board text removed: "7"
- board text removed: "8"
- board text removed: "IN"
- board text removed: "MIDI"

Commit message: ..
Routing:
- net +5V: track 73.5 -> 117.1 mm, vias 0 -> 5
- net MIDI_4_RX: track 74.2 -> 77.1 mm
- net MIDI_IN_T_3: track 79.4 -> 80.5 mm
- net MIDI_IN_T_2: track 132.4 -> 133.0 mm
- net MIDI_IN_T_4: track 104.2 -> 104.8 mm

Commit message: further tweaks
Routing:
- net +3V3: track 156.4 -> 224.0 mm, vias 1 -> 0
- net GND: track 101.7 -> 156.0 mm, vias 6 -> 10
- net MIDI_1_RX: track 84.5 -> 116.3 mm
- net +5V: track 117.1 -> 140.5 mm, vias 5 -> 7
- net MIDI_IN_T_1: track 42.7 -> 46.4 mm
- net MIDI_IN_R_4: track 93.7 -> 96.9 mm, vias 1 -> 0
- net MIDI_4_TX: track 73.9 -> 76.6 mm
- net MIDI_IN_T_3: track 80.5 -> 82.6 mm
- net Net-(ULPZWmidi4-A2): track 9.95 -> 11.5 mm
Other:
- board text added: "IN"
- board text added: "MIDI"

Commit message: cleaned up schematic a little to add the front/backboard connection
Parts:
- moved C5 64.5 mm to (218.5, 78.2), turned to -90 degrees
- moved C2 58.3 mm to (217.5, 144.0), turned to 180 degrees
- renumbered REF** to J1_BACK, REF** to J1_FRONT, REF** to J2_BACK, REF** to J2_FRONT
Routing:
- net +5V: track 140.5 -> 152.0 mm, vias 7 -> 8
- net GND: track 156.0 -> 152.6 mm, vias 10 -> 8
- net MIDI_4_TX: track 76.6 -> 74.9 mm, vias 0 -> 2
- net +3V3: track 224.0 -> 225.4 mm, vias 0 -> 1
- net MIDI_IN_R_4: track 96.9 -> 95.8 mm

Commit message: laid out quite nicely now i think
Parts:
- C2: value 100nF -> 100n
- C4: value 100n -> 100nF
- C6, R10, R12, R13, R14, R15, R16, R17, R19, R20: moved to B.Cu
- J1_BACK1: renamed from J1_BACK; value PinHeader_2x06_P2.54mm_Vertical -> Conn_02x06_Odd_Even
- J1_FRONT1: renamed from J1_FRONT; value PinSocket_2x06_P2.54mm_Vertical -> Conn_02x06_Odd_Even
- J2_BACK1: renamed from J2_BACK; value PinHeader_1x06_P2.54mm_Vertical -> Conn_01x06_Pin
- J2_FRONT1: renamed from J2_FRONT; value PinHeader_1x06_P2.54mm_Vertical -> Conn_01x06_Socket; footprint Connector_PinHeader_2.54mm:PinHeader_1x06_P2.54mm_Vertical -> Connector_PinSocket_2.54mm:PinSocket_1x06_P2.54mm_Vertical
- R1, R4, R6: moved to F.Cu
- moved C4 54.6 mm to (217.4, 152.9), turned to 180 degrees
- moved C6 52.5 mm to (217.9, 97.8), turned to -90 degrees
- moved C3 12.2 mm to (217.3, 123.2)
- moved R17 12.2 mm to (204.6, 126.8)
- moved R18 12.2 mm to (203.4, 116.0)
- moved ULPZWmidi4 12.2 mm to (209.1, 119.5)
- moved R20 12.2 mm to (214.4, 123.3)
- moved R15 6.99 mm to (204.5, 108.1)
- moved R16 6.99 mm to (202.9, 97.7)
- moved R19 6.99 mm to (215.0, 105.5)
- moved ULPZWmidi3 6.99 mm to (209.7, 101.7)
- moved C5 4.89 mm to (218.1, 83.1)
- moved R11 4.89 mm to (203.5, 89.8)
- moved R12 4.89 mm to (212.3, 92.6)
- moved R14 4.89 mm to (215.2, 90.6)
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Connections:
- C2 pad 1: +3V3 -> +5V
- C4 pad 1: +5V -> +3V3
- J1_BACK1 pad 10: MIDI_IN_T_4 -> MIDI_IN_T_4_BACK
- J1_BACK1 pad 3: MIDI_IN_R_1 -> MIDI_IN_R_1_BACK
- J1_BACK1 pad 4: MIDI_IN_T_1 -> MIDI_IN_T_1_BACK
- J1_BACK1 pad 5: MIDI_IN_R_2 -> MIDI_IN_R_2_BACK
- J1_BACK1 pad 6: MIDI_IN_T_2 -> MIDI_IN_T_2_BACK
- J1_BACK1 pad 7: MIDI_IN_R_3 -> MIDI_IN_R_3_BACK
- J1_BACK1 pad 8: MIDI_IN_T_3 -> MIDI_IN_T_3_BACK
- J1_BACK1 pad 9: MIDI_IN_R_4 -> MIDI_IN_R_4_BACK
- J1_FRONT1 pad 10: MIDI_IN_T_4 -> MIDI_IN_T_4_FRONT
- J1_FRONT1 pad 3: MIDI_IN_R_1 -> MIDI_IN_R_1_FRONT
- J1_FRONT1 pad 4: MIDI_IN_T_1 -> MIDI_IN_T_1_FRONT
- J1_FRONT1 pad 5: MIDI_IN_R_2 -> MIDI_IN_R_2_FRONT
- J1_FRONT1 pad 6: MIDI_IN_T_2 -> MIDI_IN_T_2_FRONT
- J1_FRONT1 pad 7: MIDI_IN_R_3 -> MIDI_IN_R_3_FRONT
- J1_FRONT1 pad 8: MIDI_IN_T_3 -> MIDI_IN_T_3_FRONT
- J1_FRONT1 pad 9: MIDI_IN_R_4 -> MIDI_IN_R_4_FRONT
- J2_FRONT1 pad 2: MIDI_1_TX -> MIDI_1_TX_FRONT
- J2_FRONT1 pad 3: MIDI_2_TX -> MIDI_2_TX_FRONT
- J2_FRONT1 pad 4: MIDI_3_TX -> MIDI_3_TX_FRONT
- J2_FRONT1 pad 5: MIDI_4_TX -> MIDI_4_TX_FRONT
- JMIDIIN1 pad R: MIDI_IN_R_1 -> MIDI_IN_R_1_FRONT
- JMIDIIN1 pad T: MIDI_IN_T_1 -> MIDI_IN_T_1_FRONT
- JMIDIIN2 pad R: MIDI_IN_R_3 -> MIDI_IN_R_4_FRONT
- JMIDIIN2 pad T: MIDI_IN_T_3 -> MIDI_IN_T_4_FRONT
- JMIDIIN3 pad R: MIDI_IN_R_4 -> MIDI_IN_R_3_FRONT
- JMIDIIN3 pad T: MIDI_IN_T_4 -> MIDI_IN_T_3_FRONT
- JMIDIIN4 pad R: MIDI_IN_R_2 -> MIDI_IN_R_2_FRONT
- JMIDIIN4 pad T: MIDI_IN_T_2 -> MIDI_IN_T_2_FRONT
- R10 pad 2: MIDI_IN_T_1 -> MIDI_IN_T_1_BACK
- R11 pad 2: MIDI_IN_R_3 -> MIDI_IN_R_3_BACK
- R12 pad 2: MIDI_IN_T_3 -> MIDI_IN_T_3_BACK
- R15 pad 2: MIDI_IN_R_4 -> MIDI_IN_R_4_BACK
- R16 pad 2: MIDI_IN_T_4 -> MIDI_IN_T_4_BACK
- R17 pad 2: MIDI_IN_R_2 -> MIDI_IN_R_2_BACK
- R18 pad 2: MIDI_IN_T_2 -> MIDI_IN_T_2_BACK
- R5 pad 2: MIDI_1_TX -> MIDI_1_TX_FRONT
- R6 pad 2: MIDI_2_TX -> MIDI_2_TX_FRONT
- R7 pad 2: MIDI_3_TX -> MIDI_3_TX_FRONT
- R8 pad 2: MIDI_4_TX -> MIDI_4_TX_FRONT
- R9 pad 2: MIDI_IN_R_1 -> MIDI_IN_R_1_BACK
- ULPZWmidi1 pad 2: MIDI_IN_T_1 -> MIDI_IN_T_1_BACK
- ULPZWmidi1 pad 3: MIDI_IN_R_1 -> MIDI_IN_R_1_BACK
- ULPZWmidi2 pad 2: MIDI_IN_T_3 -> MIDI_IN_T_3_BACK
- ULPZWmidi2 pad 3: MIDI_IN_R_3 -> MIDI_IN_R_3_BACK
- ULPZWmidi3 pad 2: MIDI_IN_T_4 -> MIDI_IN_T_4_BACK
- ULPZWmidi3 pad 3: MIDI_IN_R_4 -> MIDI_IN_R_4_BACK
- ULPZWmidi4 pad 2: MIDI_IN_T_2 -> MIDI_IN_T_2_BACK
- ULPZWmidi4 pad 3: MIDI_IN_R_2 -> MIDI_IN_R_2_BACK
Routing:
- net MIDI_IN_T_2: track 133.1 -> 0.00 mm
- net MIDI_IN_R_2: track 123.7 -> 0.00 mm
- net MIDI_IN_R_2_BACK: track 0.00 -> 106.5 mm
- net MIDI_IN_T_4: track 104.8 -> 0.00 mm
- net MIDI_IN_R_4: track 95.8 -> 0.00 mm
- net MIDI_IN_T_2_BACK: track 0.00 -> 88.5 mm
- net MIDI_IN_T_3: track 82.6 -> 0.00 mm
- net MIDI_IN_T_4_BACK: track 0.00 -> 65.2 mm
- net MIDI_IN_R_3: track 59.6 -> 0.00 mm
- net MIDI_IN_R_4_BACK: track 0.00 -> 59.0 mm
- net MIDI_IN_T_3_BACK: track 0.00 -> 58.9 mm
- net MIDI_IN_T_2_FRONT: track 0.00 -> 57.1 mm
- net MIDI_1_TX_FRONT: track 0.00 -> 55.2 mm
- net MIDI_1_TX: track 77.4 -> 25.2 mm
- net MIDI_4_TX: track 74.9 -> 24.8 mm, vias 2 -> 0
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Other:
- outline, holes or cut-outs redrawn
- board text added: "!!!NOT POWER!!!"

Commit message: put output jacks in correct order, added labelling to pins
Parts:
- moved R2 35.4 mm to (180.5, 120.2), turned to 0 degrees
- moved JMIDIOUT2 25.1 mm to (191.6, 126.5)
- moved JMIDIOUT4 25.1 mm to (191.5, 151.6)
- moved R4 25.1 mm to (187.7, 145.3)
- moved R8 25.1 mm to (177.0, 155.5)
- moved R7 14.8 mm to (180.3, 132.8), turned to 0 degrees
- moved R6 4.20 mm to (177.0, 130.3), turned to 90 degrees
Routing:
- net MIDI_4_TX_FRONT: track 49.2 -> 16.2 mm
- net +3V3: track 198.8 -> 177.8 mm
- net Net-(JMIDIOUT2-PadT): track 20.0 -> 5.15 mm
- net MIDI_3_TX_FRONT: track 15.6 -> 28.3 mm
- net MIDI_2_TX_FRONT: track 36.7 -> 42.7 mm
- net Net-(JMIDIOUT3-PadT): track 10.6 -> 6.04 mm
- net Net-(JMIDIOUT2-PadR): track 13.1 -> 10.6 mm
Other:
- board text added: "3v3"
- board text added: "5v"
- board text added: "LD1117"
- board text added: "gnd"
- board text added: "in"
- board text added: "out"
- board text added: "rng"
- board text added: "rx"
- board text added: "tip"
- board text added: "tx"

Commit message: screenies + jlcpcb placeholders
Other:
- board text added: "JLCPCBJLCPCBJLCPCB"
- board text added: "a century ago i'd have died, now i'm kicking"
- board text added: "tyrellcorp"
Changed lines of the file:
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@@
     (effects (font (size 1.5 1.5) (thickness 0.3) bold) (justify left bottom mirror))
+  )
+  (gr_text "JLCPCBJLCPCBJLCPCB" (at 218.694 160.3756 270) (layer "B.SilkS")
+    (effects (font (size 1 1) (thickness 0.25) bold italic) (justify left bottom mirror))
   )
   (gr_text "rx" (at 206.9084 130.7084) (layer "B.SilkS")
@@
     (effects (font (size 1.5 1.5) (thickness 0.3) bold) (justify left bottom mirror))
   )
+  (gr_text "JLCPCBJLCPCBJLCPCB" (at 175.7172 105.3592 270) (layer "B.SilkS")
+    (effects (font (size 1 1) (thickness 0.25) bold italic) (justify left bottom mirror))
+  )
   (gr_text "1" (at 205.1304 132.842) (layer "B.SilkS")
     (effects (font (size 1.5 1.5) (thickness 0.3) bold) (justify left bottom mirror))
+  )
+  (gr_text "JLCPCBJLCPCBJLCPCB" (at 226.7712 62.1792 270) (layer "B.SilkS")
+    (effects (font (size 1 1) (thickness 0.25) bold italic) (justify left bottom mirror))
   )
   (gr_text "!!!NOT POWER!!!" (at 202.184 127.9144 90) (layer "B.SilkS")
@@
   (gr_text "gnd" (at 210.1596 138.5316 90) (layer "B.SilkS")
     (effects (font (size 1.5 1.5) (thickness 0.3) bold) (justify left bottom mirror))
+  )
+  (gr_text "a century ago i'd have died, now i'm kicking" (at 243.2812 168.2496 -90) (layer "B.SilkS")
+    (effects (font (size 1.5 1.5) (thickness 0.3) bold italic) (justify left bottom mirror))
   )
   (gr_text "2" (at 207.6704 132.842) (layer "B.SilkS")
@@
     (effects (font (size 1 1) (thickness 0.15)) (justify left bottom))
   )
+  (gr_text "tyrellcorp" (at 230.0732 49.276) (layer "F.SilkS")
+    (effects (font (size 1.5 1.5) (thickness 0.3) bold italic) (justify left bottom))
+  )
   (gr_text "4\n" (at 240.2572 101.697971) (layer "F.SilkS")

Commit message: sent to jlcpcb
Parts:
- ULPZWmidi1, ULPZWmidi2, ULPZWmidi3, ULPZWmidi4: footprint Package_SO:SOIC-8_3.9x4.9mm_P1.27mm -> Package_SO:SO-8_3.9x4.9mm_P1.27mm
Routing:
- net +5V: track 130.1 -> 114.6 mm, vias 3 -> 4
- net GND: track 134.1 -> 122.4 mm, vias 6 -> 5
- net MIDI_IN_T_1_BACK: track 34.3 -> 39.1 mm
- net MIDI_IN_T_2_BACK: track 88.5 -> 90.3 mm
- net Net-(ULPZWmidi1-A1): track 4.55 -> 3.52 mm
- net MIDI_IN_R_2_BACK: track 106.5 -> 105.5 mm
- net Net-(ULPZWmidi2-A2): track 3.44 -> 2.41 mm
- net MIDI_IN_R_4_BACK: track 59.0 -> 58.0 mm
- net MIDI_3_RX: track 64.7 -> 65.7 mm
- net Net-(ULPZWmidi3-A1): track 4.56 -> 5.18 mm
- net Net-(JMIDIOUT2-PadT): track 5.15 -> 4.57 mm
