File: expander_midi/expander_midi.kicad_sch (KiCad schematic)
At the start: 73 parts

Commit message: rough layout of single midi expander
Parts:
- removed C5, C6, C7, C8: 100n, Capacitor_SMD:C_0805_2012Metric, symbol Device:C
- removed JMIDIIN5, JMIDIIN6, JMIDIIN7, JMIDIIN8, JMIDIOUT5, JMIDIOUT6, JMIDIOUT7, JMIDIOUT8: MIDI In Jack 3.5mm stereo jack, doctea:Jack_3.5mm_QingPu_WQP-PJ398SM_TRS_Vertical_CircularHoles, symbol CV12 Feb 22 with lpzw midi 5v-rescue:AudioJack3-Connector
- removed MIDI_EXPANDER_MAIN1: 20 pin header, Connector_PinHeader_2.54mm:PinHeader_2x10_P2.54mm_Vertical, symbol Connector_Generic:Conn_02x10_Counter_Clockwise
- removed R13, R14, R15, R16, R19, R20, R21, R22: 220R, Resistor_SMD:R_0805_2012Metric, symbol Device:R
- removed R17, R18, R23, R24: 470R, Resistor_SMD:R_0805_2012Metric, symbol Device:R
- removed R33, R34, R35, R36, R37, R38, R39, R40: 47R, Resistor_SMD:R_0805_2012Metric, symbol Device:R
- removed ULPZWmidi5, ULPZWmidi6, ULPZWmidi7, ULPZWmidi8: HCPL-0631, Package_SO:SOIC-8_3.9x4.9mm_P1.27mm, symbol Isolator:HCPL-0631
- added C6, C7: 100nF, Capacitor_THT:C_Axial_L5.1mm_D3.1mm_P7.50mm_Horizontal, symbol Device:C_Small
- added MIDI_EXPANDER_1: Conn_02x05_Counter_Clockwise, Connector_PinHeader_2.54mm:PinHeader_2x05_P2.54mm_Vertical, symbol Connector_Generic:Conn_02x05_Counter_Clockwise
- added U1: LD1117, Package_TO_SOT_SMD:SOT-223-3_TabPin2, symbol Regulator_Linear:LD1117S33TR_SOT223
- C3: renamed from C1; footprint Capacitor_SMD:C_0805_2012Metric -> Capacitor_THT:C_Axial_L5.1mm_D3.1mm_P7.50mm_Horizontal
- C4: renamed from C3; footprint Capacitor_SMD:C_0805_2012Metric -> Capacitor_THT:C_Axial_L5.1mm_D3.1mm_P7.50mm_Horizontal
- C5: renamed from C4; footprint Capacitor_SMD:C_0805_2012Metric -> Capacitor_THT:C_Axial_L5.1mm_D3.1mm_P7.50mm_Horizontal
- C6: renamed from C2; footprint Capacitor_SMD:C_0805_2012Metric -> Capacitor_THT:C_Axial_L5.1mm_D3.1mm_P7.50mm_Horizontal
- R1: renamed from R31; footprint Resistor_SMD:R_0805_2012Metric -> Resistor_THT:R_Axial_DIN0207_L6.3mm_D2.5mm_P7.62mm_Horizontal
- R10: renamed from R2; footprint Resistor_SMD:R_0805_2012Metric -> Resistor_THT:R_Axial_DIN0207_L6.3mm_D2.5mm_P7.62mm_Horizontal
- R11: renamed from R7; footprint Resistor_SMD:R_0805_2012Metric -> Resistor_THT:R_Axial_DIN0207_L6.3mm_D2.5mm_P7.62mm_Horizontal
- R12: renamed from R8; footprint Resistor_SMD:R_0805_2012Metric -> Resistor_THT:R_Axial_DIN0207_L6.3mm_D2.5mm_P7.62mm_Horizontal
- R13: renamed from R3; footprint Resistor_SMD:R_0805_2012Metric -> Resistor_THT:R_Axial_DIN0207_L6.3mm_D2.5mm_P7.62mm_Horizontal
- R14: renamed from R9; footprint Resistor_SMD:R_0805_2012Metric -> Resistor_THT:R_Axial_DIN0207_L6.3mm_D2.5mm_P7.62mm_Horizontal
- R15: renamed from R10; footprint Resistor_SMD:R_0805_2012Metric -> Resistor_THT:R_Axial_DIN0207_L6.3mm_D2.5mm_P7.62mm_Horizontal
- R16: renamed from R11; footprint Resistor_SMD:R_0805_2012Metric -> Resistor_THT:R_Axial_DIN0207_L6.3mm_D2.5mm_P7.62mm_Horizontal
- R17: renamed from R4; footprint Resistor_SMD:R_0805_2012Metric -> Resistor_THT:R_Axial_DIN0207_L6.3mm_D2.5mm_P7.62mm_Horizontal
- R18: renamed from R5; footprint Resistor_SMD:R_0805_2012Metric -> Resistor_THT:R_Axial_DIN0207_L6.3mm_D2.5mm_P7.62mm_Horizontal
- R19: renamed from R12; footprint Resistor_SMD:R_0805_2012Metric -> Resistor_THT:R_Axial_DIN0207_L6.3mm_D2.5mm_P7.62mm_Horizontal
- R2: renamed from R25; footprint Resistor_SMD:R_0805_2012Metric -> Resistor_THT:R_Axial_DIN0207_L6.3mm_D2.5mm_P7.62mm_Horizontal
- R20: renamed from R6; footprint Resistor_SMD:R_0805_2012Metric -> Resistor_THT:R_Axial_DIN0207_L6.3mm_D2.5mm_P7.62mm_Horizontal
- R3: renamed from R29; footprint Resistor_SMD:R_0805_2012Metric -> Resistor_THT:R_Axial_DIN0207_L6.3mm_D2.5mm_P7.62mm_Horizontal
- R4: renamed from R27; footprint Resistor_SMD:R_0805_2012Metric -> Resistor_THT:R_Axial_DIN0207_L6.3mm_D2.5mm_P7.62mm_Horizontal
- R5: renamed from R32; footprint Resistor_SMD:R_0805_2012Metric -> Resistor_THT:R_Axial_DIN0207_L6.3mm_D2.5mm_P7.62mm_Horizontal
- R6: renamed from R26; footprint Resistor_SMD:R_0805_2012Metric -> Resistor_THT:R_Axial_DIN0207_L6.3mm_D2.5mm_P7.62mm_Horizontal
- R7: renamed from R30; footprint Resistor_SMD:R_0805_2012Metric -> Resistor_THT:R_Axial_DIN0207_L6.3mm_D2.5mm_P7.62mm_Horizontal
- R8: renamed from R28; footprint Resistor_SMD:R_0805_2012Metric -> Resistor_THT:R_Axial_DIN0207_L6.3mm_D2.5mm_P7.62mm_Horizontal
- R9: renamed from R1; footprint Resistor_SMD:R_0805_2012Metric -> Resistor_THT:R_Axial_DIN0207_L6.3mm_D2.5mm_P7.62mm_Horizontal
- renumbered JMIDIIN3 to JMIDIIN2, JMIDIIN4 to JMIDIIN3, JMIDIIN2 to JMIDIIN4, JMIDIOUT4 to JMIDIOUT1, JMIDIOUT1 to JMIDIOUT2, JMIDIOUT2 to JMIDIOUT4, ULPZWmidi3 to ULPZWmidi2, ULPZWmidi4 to ULPZWmidi3, ULPZWmidi2 to ULPZWmidi4
Connections:
- net MIDI_5_TX is gone; now on net MIDI_3_TX: R7.2
- net MIDI_7_TX is gone; now on net MIDI_1_TX: R5.2
- net +3V3: now also C7.1, U1.2 (VO)
- net +5V: now also C6.1, MIDI_EXPANDER_1.5 (Pin_5), U1.3 (VI)
- net GND: now also C6.2, C7.2, MIDI_EXPANDER_1.6 (Pin_6), U1.1 (GND)
- net MIDI_1_RX: now also MIDI_EXPANDER_1.1 (Pin_1)
- net MIDI_1_TX: now also MIDI_EXPANDER_1.2 (Pin_2); no longer R6.2
- net MIDI_2_RX: now also MIDI_EXPANDER_1.3 (Pin_3)
- net MIDI_2_TX: now also R6.2, MIDI_EXPANDER_1.4 (Pin_4)
- net MIDI_3_RX: now also MIDI_EXPANDER_1.10 (Pin_10)
- net MIDI_3_TX: now also MIDI_EXPANDER_1.9 (Pin_9); no longer R8.2
- net MIDI_4_RX: now also MIDI_EXPANDER_1.8 (Pin_8)
- net MIDI_4_TX: now also R8.2, MIDI_EXPANDER_1.7 (Pin_7)
- net MIDI_IN_T_4: now reaches JMIDIIN3.T, R16.2, ULPZWmidi3.2 (C1)
- net MIDI_IN_R_4: now reaches JMIDIIN3.R, R15.2, ULPZWmidi3.3 (C2)
- net MIDI_IN_R_1: now reaches JMIDIIN1.R, R9.2, ULPZWmidi1.3 (C2)
- net MIDI_IN_T_2: now reaches JMIDIIN4.T, R18.2, ULPZWmidi4.2 (C1)
- net MIDI_IN_R_2: now reaches JMIDIIN4.R, R17.2, ULPZWmidi4.3 (C2)
- net MIDI_IN_R_3: now reaches JMIDIIN2.R, R11.2, ULPZWmidi2.3 (C2)
- net MIDI_IN_T_3: now reaches JMIDIIN2.T, R12.2, ULPZWmidi2.2 (C1)
- net MIDI_IN_T_1: now reaches JMIDIIN1.T, R10.2, ULPZWmidi1.2 (C1)
Other:
- moved on the sheet: JMIDIIN1, JMIDIOUT1, JMIDIOUT2, JMIDIOUT3, JMIDIOUT4, R1, R2, R3, R4, R5, R6, R7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

Commit message: cleaned up schematic a little to add the front/backboard connection
Parts:
- removed C5, C6: 100n, Capacitor_THT:C_Axial_L5.1mm_D3.1mm_P7.50mm_Horizontal, symbol Device:C
- added C7, C8: 100n, Capacitor_THT:C_Axial_L5.1mm_D3.1mm_P7.50mm_Horizontal, symbol Device:C
- added J1_BACK, J1_FRONT: Conn_02x06_Odd_Even, symbol Connector_Generic:Conn_02x06_Odd_Even
- added J2_BACK: Conn_01x06_Pin, symbol Connector:Conn_01x06_Pin
- added J2_FRONT: Conn_01x06_Socket, symbol Connector:Conn_01x06_Socket
Connections:
- net +3V3: now also J1_BACK.11 (Pin_11), J1_BACK.12 (Pin_12), J1_FRONT.11 (Pin_11), J1_FRONT.12 (Pin_12), J2_BACK.6 (Pin_6), J2_FRONT.6 (Pin_6)
- net +5V: now also C7.1, C8.1
- net GND: now also C7.2, C8.2, J1_BACK.1 (Pin_1), J1_BACK.2 (Pin_2), J1_FRONT.1 (Pin_1), J1_FRONT.2 (Pin_2), J2_BACK.1 (Pin_1), J2_FRONT.1 (Pin_1)
- net MIDI_1_TX: no longer R5.2
- net MIDI_2_TX: no longer R6.2
- net MIDI_3_TX: no longer R7.2
- net MIDI_4_TX: no longer R8.2
- net MIDI_IN_R_1 renamed MIDI_IN_R_1_BACK
- net MIDI_IN_R_1_BACK: now also J1_BACK.3 (Pin_3); no longer JMIDIIN1.R
- net MIDI_IN_R_2 renamed MIDI_IN_R_2_BACK
- net MIDI_IN_R_2_BACK: now also J1_BACK.5 (Pin_5); no longer JMIDIIN4.R
- net MIDI_IN_R_3 renamed MIDI_IN_R_3_BACK
- net MIDI_IN_R_3_BACK: now also J1_BACK.7 (Pin_7); no longer JMIDIIN2.R
- net MIDI_IN_R_4 renamed MIDI_IN_R_4_BACK
- net MIDI_IN_R_4_BACK: now also J1_BACK.9 (Pin_9); no longer JMIDIIN3.R
- net MIDI_IN_T_1 renamed MIDI_IN_T_1_BACK
- net MIDI_IN_T_1_BACK: now also J1_BACK.4 (Pin_4); no longer JMIDIIN1.T
- net MIDI_IN_T_2 renamed MIDI_IN_T_2_BACK
- net MIDI_IN_T_2_BACK: now also J1_BACK.6 (Pin_6); no longer JMIDIIN4.T
- net MIDI_IN_T_3 renamed MIDI_IN_T_3_BACK
- net MIDI_IN_T_3_BACK: now also J1_BACK.8 (Pin_8); no longer JMIDIIN2.T
- net MIDI_IN_T_4 renamed MIDI_IN_T_4_BACK
- net MIDI_IN_T_4_BACK: now also J1_BACK.10 (Pin_10); no longer JMIDIIN3.T
- new net MIDI_1_TX_BACK: J2_BACK.2 (Pin_2)
- new net MIDI_1_TX_FRONT: J2_FRONT.2 (Pin_2), R5.2
- new net MIDI_2_TX_BACK: J2_BACK.3 (Pin_3)
- new net MIDI_2_TX_FRONT: J2_FRONT.3 (Pin_3), R6.2
- new net MIDI_3_TX_BACK: J2_BACK.4 (Pin_4)
- new net MIDI_3_TX_FRONT: J2_FRONT.4 (Pin_4), R7.2
- new net MIDI_4_TX_BACK: J2_BACK.5 (Pin_5)
- new net MIDI_4_TX_FRONT: J2_FRONT.5 (Pin_5), R8.2
- new net MIDI_IN_R_1_FRONT: J1_FRONT.3 (Pin_3), JMIDIIN1.R
- new net MIDI_IN_R_2_FRONT: J1_FRONT.5 (Pin_5), JMIDIIN4.R
- new net MIDI_IN_R_3_FRONT: J1_FRONT.7 (Pin_7), JMIDIIN2.R
- new net MIDI_IN_R_4_FRONT: J1_FRONT.9 (Pin_9), JMIDIIN3.R
- new net MIDI_IN_T_1_FRONT: J1_FRONT.4 (Pin_4), JMIDIIN1.T
- new net MIDI_IN_T_2_FRONT: J1_FRONT.6 (Pin_6), JMIDIIN4.T
- new net MIDI_IN_T_3_FRONT: J1_FRONT.8 (Pin_8), JMIDIIN2.T
- new net MIDI_IN_T_4_FRONT: J1_FRONT.10 (Pin_10), JMIDIIN3.T
Other:
- moved on the sheet: C4, C6, C7, JMIDIIN1, JMIDIIN2, JMIDIIN3, JMIDIIN4, JMIDIOUT1, JMIDIOUT2, JMIDIOUT3, JMIDIOUT4, MIDI_EXPANDER_1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

Commit message: laid out quite nicely now i think
Parts:
- J1_BACK1: renamed from J1_BACK; footprint (none) -> Connector_PinHeader_2.54mm:PinHeader_2x06_P2.54mm_Vertical
- J1_FRONT1: renamed from J1_FRONT; footprint (none) -> Connector_PinSocket_2.54mm:PinSocket_2x06_P2.54mm_Vertical
- J2_BACK1: renamed from J2_BACK; footprint (none) -> Connector_PinHeader_2.54mm:PinHeader_1x06_P2.54mm_Vertical
- J2_FRONT1: renamed from J2_FRONT; footprint (none) -> Connector_PinSocket_2.54mm:PinSocket_1x06_P2.54mm_Vertical
- renumbered C7 to C2, C4 to C3, C8 to C5, C3 to C6, JMIDIIN3 to JMIDIIN2, JMIDIIN2 to JMIDIIN3
Connections:
- net MIDI_1_TX_BACK is gone; now on net MIDI_1_TX: J2_BACK1.2 (Pin_2)
- net MIDI_2_TX_BACK is gone; now on net MIDI_2_TX: J2_BACK1.3 (Pin_3)
- net MIDI_3_TX_BACK is gone; now on net MIDI_3_TX: J2_BACK1.4 (Pin_4)
- net MIDI_4_TX_BACK is gone; now on net MIDI_4_TX: J2_BACK1.5 (Pin_5)
