File: usb_midi_clocker circuits.kicad_pcb (KiCad board)
At the start: 2 copper layers, 135.6 x 128.5 mm, 21 parts, among them J2 USB power, J4 USB Host header, J5 Conn_01x08_Pin, SW1 Rotary_Encoder_Switch, SW2 SW_Push_Back, SW3 SW_Push_Select, U1 L78L05_TO92, U2 Teensy4.1, U3 TFT_320x240

Commit message: laid out
Parts:
- removed MIDI expander: 20 pin header, Connector_PinHeader_2.54mm:PinHeader_2x10_P2.54mm_Vertical
- removed SPI gate expander: 16 pin header, Connector_PinHeader_2.54mm:PinHeader_2x08_P2.54mm_Vertical
- removed i2c cv expander: 8 pin header, Connector_PinHeader_2.54mm:PinHeader_2x04_P2.54mm_Vertical
- added CV_INPUT_I2C_EXPANDER_MAIN1: 8 pin header, Connector_PinHeader_2.54mm:PinHeader_2x04_P2.54mm_Vertical, B.Cu at (99.8, 87.8)
- added GATE_OUTPUT_EXPANDER1: 16 pin header, Connector_PinHeader_2.54mm:PinHeader_2x08_P2.54mm_Vertical, B.Cu at (93.8, 72.4)
- added MIDI_EXPANDER_1: Conn_02x05_Counter_Clockwise, Connector_PinHeader_2.54mm:PinHeader_2x05_P2.54mm_Vertical, B.Cu at (52.7, 92.5)
- added MIDI_EXPANDER_2: Conn_02x05_Counter_Clockwise, Connector_PinHeader_2.54mm:PinHeader_2x05_P2.54mm_Vertical, B.Cu at (52.7, 73.6)
- added R2: R, Resistor_THT:R_Axial_DIN0309_L9.0mm_D3.2mm_P2.54mm_Vertical, B.Cu at (66.7, 128.9)
- added R3: R, Resistor_THT:R_Axial_DIN0309_L9.0mm_D3.2mm_P2.54mm_Vertical, B.Cu at (66.7, 136.5)
- added R4: 100r, Resistor_THT:R_Axial_DIN0309_L9.0mm_D3.2mm_P2.54mm_Vertical, B.Cu at (70.3, 43.2)
- added R5: R, Resistor_THT:R_Axial_DIN0309_L9.0mm_D3.2mm_P2.54mm_Vertical, B.Cu at (85.5, 44.4)
- added R6: R, Resistor_THT:R_Axial_DIN0309_L9.0mm_D3.2mm_P2.54mm_Vertical, B.Cu at (64.2, 43.2)
- R1: footprint Resistor_THT:R_Axial_DIN0207_L6.3mm_D2.5mm_P10.16mm_Horizontal -> Resistor_THT:R_Axial_DIN0309_L9.0mm_D3.2mm_P2.54mm_Vertical
Connections:
- U2 pad 11: TFT DC -> TFT CS
- U2 pad 12: TFT CS -> TFT DC
- U2 pad 23: TFT Reset -> Touch IRQ
- U2 pad 24: unused_pin_24 -> unused_pin_32
- U2 pad 28: unused_pin_28 -> unused_pin_36
- U2 pad 44: Touch IRQ -> unused_pin_22
- U3 pad 4: TFT Reset -> +3V3
- U3 pad 8: +3V3 -> Net-(U3-LED)
Routing:
- net Touch IRQ: track 89.3 -> 29.0 mm
- net MIDI_6_TX: track 56.2 -> 13.5 mm
- net MIDI_1_TX: track 65.3 -> 22.8 mm, vias 0 -> 1
- net unused_pin_28: track 41.5 -> 0.00 mm, vias 1 -> 0
- net MIDI_1_RX: track 64.5 -> 27.3 mm, vias 2 -> 1
- net MIDI_8_RX: track 66.3 -> 31.5 mm, vias 0 -> 1
- net MIDI_7_RX: track 41.9 -> 12.4 mm, vias 1 -> 0
- net MIDI_6_RX: track 44.8 -> 15.3 mm, vias 1 -> 0
- net TFT Reset: track 27.2 -> 0.00 mm, vias 1 -> 0
- net MIDI_7_TX: track 41.2 -> 15.4 mm, vias 1 -> 0
- net GND: track 40.0 -> 14.4 mm, vias 2 -> 1
- net unused_pin_24: track 25.0 -> 0.00 mm, vias 1 -> 0
- net TFT DC: track 73.6 -> 54.2 mm
- net MIDI_8_TX: track 51.7 -> 33.1 mm, vias 0 -> 1
- net MIDI_2_TX: track 30.2 -> 12.2 mm, vias 2 -> 0
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
Commit message: laid out some more
Parts:
- J5: footprint doctea:PinHeader_2x04_P2.54mm_Vertical-AlternatePinNumbering -> Connector_PinHeader_2.54mm:PinHeader_2x05_P2.54mm_Vertical
- moved R1 6.07 mm to (98.7, 48.7)
- renumbered CV_INPUT_I2C_EXPANDER_MAIN1 to CV_INPUT_I2C_EXPANDER
Connections:
- J5 pad 1: unused_pin_33 -> unused_pin_36
- J5 pad 2: unused_pin_28 -> unused_pin_33
- J5 pad 3: unused_pin_24 -> unused_pin_32
- J5 pad 4: unused_pin_23 -> unused_pin_24
- J5 pad 5: +5V -> unused_pin_23
- J5 pad 6: +3V3 -> +5V
- J5 pad 7: GND -> +3V3
Routing:
- net unused_pin_36: track 0.00 -> 45.0 mm, vias 0 -> 2
- net +5V: track 240.7 -> 216.7 mm, vias 1 -> 2
- net unused_pin_23: track 116.7 -> 100.3 mm, vias 3 -> 1
- net unused_pin_32: track 0.00 -> 15.0 mm, vias 0 -> 1
- net Net-(U3-VCC): track 19.6 -> 13.1 mm
- net GND: track 14.4 -> 20.5 mm, vias 1 -> 2
- net +3V3: track 241.0 -> 237.2 mm
- net INT_2: track 25.0 -> 22.4 mm, vias 1 -> 0
- net unused_pin_33: track 29.9 -> 28.6 mm
- net External CS1: track 12.2 -> 11.6 mm, vias 1 -> 0
- net MIDI_2_TX: track 12.2 -> 11.6 mm
- net INT_1: track 22.8 -> 22.6 mm, vias 1 -> 0
- net MIDI_1_TX: track 22.8 -> 22.9 mm, vias 1 -> 2
- net External CS2: vias 1 -> 0
- net Net-(U2-5_IN2): vias 1 -> 0
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Other:
- board text added: "23"
- board text added: "24"
- board text added: "32"
- board text added: "33"
- board text added: "36"
- board text added: "gnd"
- board text added: "nc"
- board text removed: "pin 23"
- board text removed: "pin 24"
- board text removed: "pin 28"
- board text removed: "pin 33"

Commit message: updated files
Routing:
- net +5V: track 216.7 -> 219.1 mm
- net unused_pin_23: vias 1 -> 2
Other:
- board text added: "JLCPCBJLCPCBJLCPCB"
- board text added: "and it tastes good"
- board text added: "castles crumble in landslides, and i munch the rubble"
Changed lines of the file:
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@@
     (effects (font (size 1 1) (thickness 0.15)) (justify mirror))
+  )
+  (gr_text "JLCPCBJLCPCBJLCPCB" (at 157.48 151.2824) (layer "B.SilkS")
+    (effects (font (size 1 1) (thickness 0.25) bold) (justify left bottom mirror))
   )
   (gr_text "+5v\n" (at 52.7558 41.9608 90) (layer "B.SilkS")
@@
     (effects (font (size 1 1) (thickness 0.15)) (justify mirror))
   )
+  (gr_text "and it tastes good" (at 156.1592 33.9852) (layer "B.SilkS")
+    (effects (font (size 1 1) (thickness 0.25) bold) (justify left bottom mirror))
+  )
   (gr_text "stripe" (at 97.3582 88.646) (layer "B.SilkS" knockout)
     (effects (font (size 1 1) (thickness 0.15)) (justify left bottom mirror))
@@
   (gr_text "SDA" (at 96.3676 80.137) (layer "B.SilkS")
     (effects (font (size 1 1) (thickness 0.15)) (justify mirror))
+  )
+  (gr_text "castles crumble in landslides, and i munch the rubble" (at 96.0628 36.1696) (layer "B.SilkS")
+    (effects (font (size 1 1) (thickness 0.25) bold) (justify left bottom mirror))
   )
   (gr_text "+3v3\n" (at 50.0634 50.5714 90) (layer "B.SilkS")
@@
     )
   )
+  (gr_text "JLCPCBJLCPCBJLCPCB" (at 44.2722 34.8742 -90) (layer "F.SilkS")
+    (effects (font (size 1 1) (thickness 0.25) bold) (justify left bottom))
+  )
   (gr_text "<< back" (at 143.0274 124.9172 -90) (layer "F.SilkS")
     (effects (font (size 1.5 1.5) (thickness 0.3) bold) (justify left bottom))
   )
   (segment (start 100.9716 84.0674) (end 94.583 84.0674) (width 0.25) (layer "F.Cu") (net 1))
+  (segment (start 50.0634 68.9864) (end 50.5206 68.5292) (width 0.25) (layer "F.Cu") (net 1))
+  (segment (start 52.705 87.4014) (end 51.5046 86.201) (width 0.25) (layer "F.Cu") (net 1))
   (segment (start 94.3356 83.82) (end 94.0562 84.0994) (width 0.25) (layer "F.Cu") (net 1))
+  (segment (start 50.0634 77.6986) (end 50.0634 68.9864) (width 0.25) (layer "F.Cu") (net 1))
   (segment (start 94.0562 91.9134) (end 94.0562 84.0994) (width 0.25) (layer "F.Cu") (net 1))
   (segment (start 99.5172 70.612) (end 99.5172 74.3712) (width 0.25) (layer "F.Cu") (net 1))
-  (segment (start 51.5046 86.201) (end 51.5046 69.7042) (width 0.25) (layer "F.Cu") (net 1))
-  (segment (start 51.5046 69.7042) (end 52.6796 68.5292) (width 0.25) (layer "F.Cu") (net 1))
+  (segment (start 50.5206 68.5292) (end 52.6796 68.5292) (width 0.25) (layer "F.Cu") (net 1))
   (segment (start 99.5172 74.3712) (end 94.3356 79.5528) (width 0.25) (layer "F.Cu") (net 1))
+  (segment (start 51.5046 86.201) (end 51.5046 79.1398) (width 0.25) (layer "F.Cu") (net 1))
   (segment (start 94.0562 91.9134) (end 87.3506 98.619) (width 0.25) (layer "F.Cu") (net 1))
-  (segment (start 52.705 87.4014) (end 51.5046 86.201) (width 0.25) (layer "F.Cu") (net 1))
   (segment (start 102.3112 80.1878) (end 102.3112 82.7278) (width 0.25) (layer "F.Cu") (net 1))
   (segment (start 102.3366 82.7024) (end 100.9716 84.0674) (width 0.25) (layer "F.Cu") (net 1))
@@
   (segment (start 52.705 87.4014) (end 47.4472 92.6592) (width 0.25) (layer "F.Cu") (net 1))
   (segment (start 94.583 84.0674) (end 94.3356 83.82) (width 0.25) (layer "F.Cu") (net 1))
+  (segment (start 51.5046 79.1398) (end 50.0634 77.6986) (width 0.25) (layer "F.Cu") (net 1))
   (segment (start 47.4472 92.6592) (end 47.4472 93.2688) (width 0.25) (layer "F.Cu") (net 1))
   (via (at 47.4472 93.2688) (size 0.8) (drill 0.4) (layers "F.Cu" "B.Cu") (net 1))
@@
   (segment (start 57.658 44.958) (end 68.6562 44.958) (width 0.25) (layer "F.Cu") (net 67))
   (segment (start 49.0982 50.9778) (end 52.578 47.498) (width 0.25) (layer "F.Cu") (net 69))
+  (segment (start 72.9996 104.7496) (end 82.55 104.7496) (width 0.25) (layer "F.Cu") (net 69))
   (segment (start 49.0982 51.0794) (end 49.0982 50.9778) (width 0.25) (layer "F.Cu") (net 69))
   (via (at 49.0982 51.0794) (size 0.8) (drill 0.4) (layers "F.Cu" "B.Cu") (net 69))
+  (via (at 72.9996 104.7496) (size 0.8) (drill 0.4) (layers "F.Cu" "B.Cu") (net 69))
   (segment (start 64.7446 104.0384) (end 56.576501 104.0384) (width 0.25) (layer "B.Cu") (net 69))
   (segment (start 67.775991 105.8746) (end 66.5808 105.8746) (width 0.25) (layer "B.Cu") (net 69))
-  (segment (start 82.55 104.7496) (end 68.900991 104.7496) (width 0.25) (layer "B.Cu") (net 69))
   (segment (start 56.576501 104.0384) (end 50.829501 109.7854) (width 0.25) (layer "B.Cu") (net 69))
   (segment (start 49.0982 109.027501) (end 49.0982 51.0794) (width 0.25) (layer "B.Cu") (net 69))
   (segment (start 49.856099 109.7854) (end 49.0982 109.027501) (width 0.25) (layer "B.Cu") (net 69))
+  (segment (start 68.900991 104.7496) (end 72.9996 104.7496) (width 0.25) (layer "B.Cu") (net 69))
   (segment (start 66.5808 105.8746) (end 64.7446 104.0384) (width 0.25) (layer "B.Cu") (net 69))
   (segment (start 68.900991 104.7496) (end 67.775991 105.8746) (width 0.25) (layer "B.Cu") (net 69))

Commit message: solve a couple of problems on main board + main panel
Parts:
- removed CV_INPUT_I2C_EXPANDER: 8 pin header, Connector_PinHeader_2.54mm:PinHeader_2x04_P2.54mm_Vertical
- removed U1: L78L05_TO92, Package_TO_SOT_THT:TO-92_Inline
- added I2C_EXPANDER: 8 pin header, Connector_PinHeader_2.54mm:PinHeader_2x04_P2.54mm_Vertical, B.Cu at (99.8, 87.8)
- added U4: L7805, Package_TO_SOT_THT:TO-220-3_Vertical, B.Cu at (87.8, 97.0)
- C6: value 10uF -> 330nF
- C7: value 1uF -> 100nF
- J5: value Conn_01x08_Pin -> Conn_01x09_Pin
- moved C7 16.2 mm to (94.3, 84.0), turned to 180 degrees
Routing:
- net GND: track 20.5 -> 10.5 mm, vias 2 -> 1
- net INT_2: track 22.4 -> 29.7 mm
- net +12V: track 22.2 -> 27.8 mm
- net TFT SPI MISO: track 62.0 -> 66.8 mm, vias 1 -> 0
- net MIDI_6_TX: track 13.5 -> 17.9 mm, vias 1 -> 0
- net INT_1: track 22.6 -> 26.3 mm
- net i2c SCL: track 28.9 -> 26.1 mm
- net Gate SPI SCK: track 31.9 -> 29.5 mm, vias 1 -> 0
- net +3V3: track 237.2 -> 239.2 mm, vias 1 -> 2
- net TFT DC: track 54.2 -> 52.5 mm
- net +5V: track 219.1 -> 218.0 mm
- net Touch IRQ: track 29.0 -> 29.6 mm
- net Gate SPI MISO: track 11.9 -> 11.6 mm, vias 1 -> 0
- net Gate SPI MOSI: track 28.0 -> 28.3 mm, vias 2 -> 0
Other:
- outline, holes or cut-outs redrawn
- board text added: "rev 2"
