File: expander_usb_sd/expander_usb_sd.kicad_pcb (KiCad board)
At the start: 2 copper layers, 59.7 x 128.5 mm, 10 parts, among them J1 Micro_SD_Card_Det1, J1-TeensyPower1 USB power - Teensy device, J2 Internal_USB_Host_Teensy, J2-USBHostPower1 USB power - host, J5-TeensyMicroUSB1 USB 5 pin to Teensy/MicroUSB, J6-USBHost1 USB 5 pin to frontpanel/Type C

Commit message: updated to correct(?) footprint + 3d model for the usb socket
Parts:
- External_USB_A_Host1: footprint Connector_USB:USB_A_Molex_105057_Vertical -> usba1vsb6:ONSHORE_USB-A1VSB6
- moved External_USB_A_Host1 4.24 mm to (128.7, 66.7), turned to -90 degrees
- moved J2-USBHostPower1 0.81 mm to (128.7, 77.0)
- renumbered J5-TeensyMicroUSB1 to J5-TeensyMicroUSB-C, J6-USBHost1 to J6-USBHost1-A, SD_connector1 to SD
Connections:
- J2 pad 5: GND -> Net-(External_USB_A_Host1-GND)
- J2-USBHostPower1 pad 2: Net-(External_USB_A_Host1-VBUS) -> Net-(External_USB_A_Host1-VUSB)
Routing:
- net GND: track 19.6 -> 4.29 mm, vias 3 -> 2
- net Net-(External_USB_A_Host1-GND): track 22.5 -> 35.3 mm
- net Net-(External_USB_A_Host1-VBUS): track 8.70 -> 0.00 mm
- net Net-(External_USB_A_Host1-D+): track 17.6 -> 22.6 mm
- net Net-(J2-Pin_1): track 3.44 -> 4.04 mm

Commit message: update labling
Parts:
- renumbered J5-TeensyMicroUSB-C to TeensyMicroUSB-C, J1-TeensyPower1 to TeensyPower, J6-USBHost1-A to USBHost-A
Routing:
- net GND: track 4.29 -> 0.04 mm
Other:
- board text added: "Pin 1"
Changed lines of the file:
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@@
     (property "ki_keywords" "connector")
     (attr through_hole)
-    (fp_text reference "J1-TeensyPower1" (at 0 2.33 90) (layer "B.SilkS")
+    (fp_text reference "TeensyPower" (at 2.55 -1.425 180) (layer "B.SilkS")
         (effects (font (size 1 1) (thickness 0.15)) (justify mirror))
     )
@@
     (property "ki_keywords" "connector")
     (attr through_hole)
-    (fp_text reference "SD" (at 1.27 2.33) (layer "B.SilkS")
+    (fp_text reference "SD" (at 1.5 -9.85) (layer "B.SilkS")
         (effects (font (size 1 1) (thickness 0.15)) (justify mirror))
     )
@@
     (property "ki_keywords" "connector")
     (attr through_hole)
-    (fp_text reference "J6-USBHost1-A" (at 1.930954 -5.94 90) (layer "B.SilkS")
+    (fp_text reference "USBHost-A" (at 1.930954 -5.94 90) (layer "B.SilkS")
         (effects (font (size 1 1) (thickness 0.15)) (justify mirror))
     )
@@
     (property "ki_keywords" "connector")
     (attr through_hole)
-    (fp_text reference "J5-TeensyMicroUSB-C" (at -2.119046 -5.84 90) (layer "B.SilkS")
+    (fp_text reference "TeensyMicroUSB-C" (at -2.119046 -5.84 90) (layer "B.SilkS")
         (effects (font (size 1 1) (thickness 0.15)) (justify mirror))
     )
@@
   (gr_arc (start 79.8 165.2) (mid 78.2 163.6) (end 79.8 162)
     (stroke (width 0.05) (type solid)) (layer "Edge.Cuts"))
+  (gr_text "Pin 1" (at 130.9 111.95) (layer "B.SilkS")
+    (effects (font (size 1 1) (thickness 0.15)) (justify left bottom mirror))
+  )
+  (gr_text "Pin 1" (at 130.8 80.2) (layer "B.SilkS")
+    (effects (font (size 1 1) (thickness 0.15)) (justify left bottom mirror))
+  )
   (gr_text "JLCPCBJLCPCBJLCPCBJLCPCB" (at 77.3 93.7 90) (layer "B.SilkS")
     (effects (font (size 1.5 1.5) (thickness 0.3) bold) (justify left bottom mirror))
@@
   (segment (start 126.583299 79.135) (end 124.85 77.401701) (width 0.25) (layer "F.Cu") (net 3))
   (segment (start 124.85 77.401701) (end 124.85 73.05) (width 0.25) (layer "F.Cu") (net 3))
+  (segment (start 130.155 79.135) (end 126.583299 79.135) (width 0.25) (layer "F.Cu") (net 3))
+  (segment (start 130.25 67.65) (end 131.65 67.65) (width 0.25) (layer "F.Cu") (net 3))
+  (segment (start 132.4 81.38) (end 130.155 79.135) (width 0.25) (layer "F.Cu") (net 3))
   (segment (start 124.85 73.05) (end 130.25 67.65) (width 0.25) (layer "F.Cu") (net 3))
-  (segment (start 130.155 79.135) (end 126.583299 79.135) (width 0.25) (layer "F.Cu") (net 3))
-  (segment (start 132.4 81.38) (end 130.155 79.135) (width 0.25) (layer "F.Cu") (net 3))
-  (segment (start 130.25 67.65) (end 131.65 67.65) (width 0.25) (layer "F.Cu") (net 3))
   (segment (start 133.7 85.16) (end 133.7 72.2) (width 0.25) (layer "F.Cu") (net 4))
   (segment (start 133.7 72.2) (end 131.65 70.15) (width 0.25) (layer "F.Cu") (net 4))
@@
   (segment (start 129.9 97.004578) (end 128.576577 98.328001) (width 0.25) (layer "B.Cu") (net 9))
   (segment (start 124.928001 97.228001) (end 124.9 97.2) (width 0.25) (layer "F.Cu") (net 10))
-  (segment (start 129.775 83.835) (end 129.775 79.585) (width 0.25) (layer "F.Cu") (net 10))
   (via (at 124.9 97.2) (size 0.8) (drill 0.4) (layers "F.Cu" "B.Cu") (net 10))
   (via (at 132.5 89.2) (size 0.8) (drill 0.4) (layers "F.Cu" "B.Cu") (net 10))

Commit message: fucking connect the USB Host pins that were completely unconnected previously... facepalm!
Parts:
- removed SD: Conn_02x04_Odd_Even, Connector_PinHeader_2.54mm:PinHeader_2x04_P2.54mm_Vertical
- removed TeensyMicroUSB-C: USB 5 pin to Teensy/MicroUSB, Connector_PinHeader_2.54mm:PinHeader_1x05_P2.54mm_Vertical
- removed TeensyPower: USB power - Teensy device, Connector_PinHeader_2.54mm:PinHeader_1x02_P2.54mm_Vertical
- removed USBHost-A: USB 5 pin to frontpanel/Type C, Connector_PinHeader_2.54mm:PinHeader_1x05_P2.54mm_Vertical
- added J1-TeensyPower1: USB power - Teensy device, Connector_PinHeader_2.54mm:PinHeader_1x02_P2.54mm_Vertical, F.Cu at (130.5, 108.3)
- added J5-TeensyMicroUSB1: USB 5 pin to Teensy/MicroUSB, Connector_PinHeader_2.54mm:PinHeader_1x05_P2.54mm_Vertical, F.Cu at (131.5, 114.2)
- added J6-USBHost1: USB 5 pin to frontpanel/Type C, Connector_PinHeader_2.54mm:PinHeader_1x05_P2.54mm_Vertical, F.Cu at (126.8, 114.2)
- added SD_connector1: Conn_02x04_Odd_Even, Connector_PinHeader_2.54mm:PinHeader_2x04_P2.54mm_Vertical, B.Cu at (128.6, 81.5)
Routing:
- net Net-(J1-TeensyPower1-Pin_1): track 0.00 -> 6.25 mm
- net Net-(J5-TeensyMicroUSB1-Pin_4): track 0.00 -> 4.70 mm
- net Net-(J5-TeensyMicroUSB1-Pin_2): track 0.00 -> 4.70 mm
- net Net-(J5-TeensyMicroUSB1-Pin_5): track 0.00 -> 4.70 mm
- net Net-(J5-TeensyMicroUSB1-Pin_3): track 0.00 -> 4.70 mm
Other:
- outline, holes or cut-outs redrawn
- board text added: ":)"
- board text added: "USB host"
- board text removed: "USBhost"

Commit message: flip headers back to correct side of board
Parts:
- J1-TeensyPower1, J5-TeensyMicroUSB1, J6-USBHost1: moved to B.Cu
- turned J1-TeensyPower1 to 90 degrees
- turned J5-TeensyMicroUSB1 to 180 degrees
- turned J6-USBHost1 to 180 degrees

Commit message: some improved routing
Routing:
- net Net-(External_USB_A_Host1-GND): track 35.3 -> 20.2 mm
- net Net-(External_USB_A_Host1-D+): track 22.6 -> 15.1 mm
Changed lines of the file:
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@@
     )
   )
-  (segment (start 131.225 71.194368) (end 130.6 70.569368) (width 0.25) (layer "B.Cu") (net 2))
-  (segment (start 130.6 70.569368) (end 130.6 66.7) (width 0.25) (layer "B.Cu") (net 2))
-  (segment (start 131.225 77.665) (end 131.225 71.194368) (width 0.25) (layer "B.Cu") (net 2))
+  (segment (start 131.225 72.075) (end 130.6 71.45) (width 0.25) (layer "B.Cu") (net 2))
+  (segment (start 131.225 77.665) (end 131.225 72.075) (width 0.25) (layer "B.Cu") (net 2))
+  (segment (start 132.4 78.84) (end 131.225 77.665) (width 0.25) (layer "B.Cu") (net 2))
   (segment (start 130.6 66.7) (end 131.65 65.65) (width 0.25) (layer "B.Cu") (net 2))
-  (segment (start 132.4 78.84) (end 131.225 77.665) (width 0.25) (layer "B.Cu") (net 2))
-  (segment (start 126.583299 79.135) (end 124.85 77.401701) (width 0.25) (layer "F.Cu") (net 3))
-  (segment (start 124.85 77.401701) (end 124.85 73.05) (width 0.25) (layer "F.Cu") (net 3))
-  (segment (start 130.155 79.135) (end 126.583299 79.135) (width 0.25) (layer "F.Cu") (net 3))
-  (segment (start 130.25 67.65) (end 131.65 67.65) (width 0.25) (layer "F.Cu") (net 3))
-  (segment (start 132.4 81.38) (end 130.155 79.135) (width 0.25) (layer "F.Cu") (net 3))
-  (segment (start 124.85 73.05) (end 130.25 67.65) (width 0.25) (layer "F.Cu") (net 3))
+  (segment (start 130.6 71.45) (end 130.6 66.7) (width 0.25) (layer "B.Cu") (net 2))
+  (segment (start 133.7 80.08) (end 133.7 69.7) (width 0.25) (layer "B.Cu") (net 3))
+  (segment (start 133.7 69.7) (end 131.65 67.65) (width 0.25) (layer "B.Cu") (net 3))
+  (segment (start 132.4 81.38) (end 133.7 80.08) (width 0.25) (layer "B.Cu") (net 3))
   (segment (start 133.7 85.16) (end 133.7 72.2) (width 0.25) (layer "F.Cu") (net 4))
   (segment (start 133.7 72.2) (end 131.65 70.15) (width 0.25) (layer "F.Cu") (net 4))
   (segment (start 132.4 86.46) (end 133.7 85.16) (width 0.25) (layer "F.Cu") (net 4))
   (segment (start 132.4 83.92) (end 132.4 86.46) (width 0.25) (layer "B.Cu") (net 4))
-  (segment (start 133.575 72.075) (end 131.65 70.15) (width 0.25) (layer "B.Cu") (net 4))
-  (segment (start 133.575 82.745) (end 133.575 72.075) (width 0.25) (layer "B.Cu") (net 4))
-  (segment (start 132.4 83.92) (end 133.575 82.745) (width 0.25) (layer "B.Cu") (net 4))
   (segment (start 127.929999 102.728) (end 126.823801 102.728) (width 0.25) (layer "B.Cu") (net 5))
   (segment (start 126 101.904199) (end 126 89.38) (width 0.25) (layer "B.Cu") (net 5))

Commit message: fixed yet more dumb routing errors on the usb_sd; probably still isn't ready to use
Parts:
- removed J2-USBHostPower1: USB power - host, Connector_PinHeader_2.54mm:PinHeader_1x02_P2.54mm_Vertical
- added USBHostPower1: USB power - host, Connector_PinHeader_2.54mm:PinHeader_1x02_P2.54mm_Vertical, F.Cu at (128.7, 77.0)
Connections:
- J2 pad 4: Net-(External_USB_A_Host1-GND) -> Net-(External_USB_A_Host1-SHIELD)
- J2 pad 5: Net-(External_USB_A_Host1-GND) -> Net-(External_USB_A_Host1-SHIELD)
Routing:
- net Net-(External_USB_A_Host1-VBUS): track 0.00 -> 16.2 mm

Commit message: believe fixed problems with expander_usb_sd; tracked a bunch of stuff that was untracked (expander_cv_output?)
Connections:
- J2 pad 4: Net-(External_USB_A_Host1-SHIELD) -> Net-(External_USB_A_Host1-GND)
- J2 pad 5: Net-(External_USB_A_Host1-SHIELD) -> Net-(External_USB_A_Host1-GND)
Routing:
- net /CMD: track 30.7 -> 33.1 mm
- net Net-(External_USB_A_Host1-GND): track 20.2 -> 22.1 mm
- net /DAT1: track 17.6 -> 18.6 mm
Changed lines of the file:
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@@
 	(net 19 "Net-(J5-TeensyMicroUSB1-Pin_4)")
 	(net 20 "Net-(J5-TeensyMicroUSB1-Pin_5)")
-	(net 21 "Net-(External_USB_A_Host1-SHIELD)")
 	(footprint "footprints:PJS008U-3000-0"
 		(layer "F.Cu")
@@
 		(tags "Through hole pin header THT 1x05 2.54mm single row")
 		(property "Reference" "J5-TeensyMicroUSB1"
-			(at 0 2.33 0)
+			(at -2 -4.6 90)
 			(layer "B.SilkS")
 			(effects
@@
 		(tags "Through hole pin header THT 1x02 2.54mm single row")
 		(property "Reference" "J1-TeensyPower1"
-			(at 0 2.33 90)
+			(at -1.975 0.01 180)
 			(layer "B.SilkS")
 			(effects
@@
 		(tags "Through hole pin header THT 1x05 2.54mm single row")
 		(property "Reference" "J6-USBHost1"
-			(at 0 2.33 0)
+			(at 1.925 -4.99 90)
 			(layer "B.SilkS")
 			(effects
@@
 			(layers "*.Cu" "*.Mask")
 			(remove_unused_layers no)
-			(net 21 "Net-(External_USB_A_Host1-SHIELD)")
+			(net 4 "Net-(External_USB_A_Host1-GND)")
 			(pinfunction "Pin_4")
 			(pintype "passive")
@@
 			(layers "*.Cu" "*.Mask")
 			(remove_unused_layers no)
-			(net 21 "Net-(External_USB_A_Host1-SHIELD)")
+			(net 4 "Net-(External_USB_A_Host1-GND)")
 			(pinfunction "Pin_5")
 			(pintype "passive")
@@
 		(tags "Through hole pin header THT 2x04 2.54mm double row")
 		(property "Reference" "SD_connector1"
-			(at 1.27 2.33 0)
+			(at 7.39 2.025 0)
 			(layer "B.SilkS")
 			(effects
@@
 	)
 	(segment
-		(start 131.225 72.075)
-		(end 130.6 71.45)
+		(start 130.2 71.05)
+		(end 130.2 67.1)
 		(width 0.25)
 		(layer "B.Cu")
@@
 	)
 	(segment
-		(start 131.225 77.665)
-		(end 131.225 72.075)
+		(start 131 77.44)
+		(end 131 71.85)
 		(width 0.25)
 		(layer "B.Cu")
@@
 	(segment
 		(start 132.4 78.84)
-		(end 131.225 77.665)
+		(end 131 77.44)
 		(width 0.25)
 		(layer "B.Cu")
@@
 	)
 	(segment
-		(start 130.6 66.7)
+		(start 130.2 67.1)
 		(end 131.65 65.65)
 		(width 0.25)
@@
 	)
 	(segment
-		(start 130.6 71.45)
-		(end 130.6 66.7)
+		(start 131 71.85)
+		(end 130.2 71.05)
 		(width 0.25)
 		(layer "B.Cu")
@@
 	)
 	(segment
-		(start 133.7 85.16)
+		(start 133.7 82.625)
 		(end 133.7 72.2)
 		(width 0.25)
@@
 	)
 	(segment
+		(start 133.7 85.16)
+		(end 133.7 82.625)
+		(width 0.25)
+		(layer "F.Cu")
+		(net 4)
+	)
+	(segment
+		(start 133.7 85.16)
+		(end 132.4 86.46)
+		(width 0.25)
+		(layer "F.Cu")
+		(net 4)
+	)
+	(segment
 		(start 133.7 72.2)
 		(end 131.65 70.15)
@@
 	)
 	(segment
-		(start 132.4 86.46)
-		(end 133.7 85.16)
+		(start 132.4 83.92)
+		(end 133.695 82.625)
+		(width 0.25)
+		(layer "F.Cu")
+		(net 4)
+	)
+	(segment
+		(start 133.695 82.625)
+		(end 133.7 82.625)
 		(width 0.25)
 		(layer "F.Cu")
@@
 	)
 	(segment
-		(start 124.885 94.189199)
-		(end 124.885 82.875)
+		(start 127.929999 96.128001)
+		(end 126.823802 96.128001)
 		(width 0.25)
 		(layer "F.Cu")
@@
 	)
 	(segment
-		(start 124.885 82.875)
+		(start 124.6 83.16)
 		(end 126.06 81.7)
 		(width 0.25)
@@
 	)
 	(segment
-		(start 126.823802 96.128001)
-		(end 124.885 94.189199)
+		(start 124.6 93.904199)
+		(end 124.6 83.16)
 		(width 0.25)
 		(layer "F.Cu")
@@
 	)
 	(segment
-		(start 127.929999 96.128001)
-		(end 126.823802 96.128001)
+		(start 126.823802 96.128001)
+		(end 124.6 93.904199)
 		(width 0.25)
 		(layer "F.Cu")
@@
 	)
 	(segment
-		(start 131.9838 99.8162)
-		(end 131.9838 91.042099)
+		(start 130.725 89.783299)
+		(end 130.725 86.325)
 		(width 0.25)
 		(layer "F.Cu")
@@
 	)
 	(segment
-		(start 126.047799 101.1624)
-		(end 126.047799 102.147799)
+		(start 126.925 103.825)
+		(end 128.475 103.825)
 		(width 0.25)
 		(layer "F.Cu")
@@
 	)
 	(segment
-		(start 131.9838 91.042099)
-		(end 131.225 90.283299)
+		(start 132.6 91.658299)
+		(end 130.725 89.783299)
 		(width 0.25)
 		(layer "F.Cu")
@@
 	)
 	(segment
-		(start 131.225 86.825)
-		(end 129.9 85.5)
+		(start 129.75 85.35)
+		(end 127.49 85.35)
 		(width 0.25)
 		(layer "F.Cu")
@@
 	)
 	(segment
-		(start 128.2898 103.5102)
-		(end 131.9838 99.8162)
+		(start 125.525 102.425)
+		(end 126.925 103.825)
 		(width 0.25)
 		(layer "F.Cu")
@@
 	)
 	(segment
-		(start 127.929999 100.527999)
-		(end 126.6822 100.527999)
+		(start 126.197001 100.527999)
+		(end 125.525 101.2)
 		(width 0.25)
 		(layer "F.Cu")
@@
 	)
 	(segment
-		(start 126.047799 102.147799)
-		(end 127.4102 103.5102)
+		(start 132.6 99.7)
+		(end 132.6 91.658299)
 		(width 0.25)
 		(layer "F.Cu")
@@
 	)
 	(segment
-		(start 129.9 85.5)
-		(end 127.34 85.5)
+		(start 125.525 101.2)
+		(end 125.525 102.425)
 		(width 0.25)
 		(layer "F.Cu")
@@
 	)
 	(segment
-		(start 127.34 85.5)
-		(end 126.06 86.78)
+		(start 128.475 103.825)
+		(end 132.6 99.7)
 		(width 0.25)
 		(layer "F.Cu")
@@
 	)
 	(segment
-		(start 126.6822 100.527999)
-		(end 126.047799 101.1624)
+		(start 127.929999 100.527999)
+		(end 126.197001 100.527999)
 		(width 0.25)
 		(layer "F.Cu")
@@
 	)
 	(segment
-		(start 131.225 90.283299)
-		(end 131.225 86.825)
+		(start 127.49 85.35)
+		(end 126.06 86.78)
 		(width 0.25)
 		(layer "F.Cu")
@@
 	)
 	(segment
-		(start 127.4102 103.5102)
-		(end 128.2898 103.5102)
+		(start 130.725 86.325)
+		(end 129.75 85.35)
 		(width 0.25)
 		(layer "F.Cu")
@@
 	)
 	(segment
-		(start 129.9 86.4)
-		(end 129.9 97.004578)
+		(start 129.25 85.35)
+		(end 129.9 86)
 		(width 0.25)
 		(layer "B.Cu")
@@
 	)
 	(segment
-		(start 128.576577 98.328001)
-		(end 127.929999 98.328001)
+		(start 129.9 86)
+		(end 129.9 97.004578)
 		(width 0.25)
 		(layer "B.Cu")
@@
 	)
 	(segment
-		(start 127.37 85.55)
-		(end 129.05 85.55)
+		(start 129.9 97.004578)
+		(end 128.576577 98.328001)
 		(width 0.25)
 		(layer "B.Cu")
@@
 	)
 	(segment
-		(start 126.06 84.24)
-		(end 127.37 85.55)
+		(start 127.17 85.35)
+		(end 129.25 85.35)
 		(width 0.25)
 		(layer "B.Cu")
@@
 	)
 	(segment
-		(start 129.05 85.55)
-		(end 129.9 86.4)
+		(start 128.576577 98.328001)
+		(end 127.929999 98.328001)
 		(width 0.25)
 		(layer "B.Cu")
@@
 	)
 	(segment
-		(start 129.9 97.004578)
-		(end 128.576577 98.328001)
+		(start 126.06 84.24)
+		(end 127.17 85.35)
 		(width 0.25)
 		(layer "B.Cu")
@@
 	)
 	(segment
-		(start 127.287199 94.5708)
-		(end 126.829999 95.028)
+		(start 127.1 87.9)
+		(end 127.325 88.125)
 		(width 0.25)
 		(layer "B.Cu")
@@
 	)
 	(segment
-		(start 126.501701 88.1)
-		(end 127.287199 88.885498)
+		(start 127.325 94.532999)
+		(end 126.829999 95.028)
 		(width 0.25)
 		(layer "B.Cu")
@@
 	)
 	(segment
-		(start 128.6 81.7)
-		(end 127.3 83)
+		(start 125.35 82.8)
+		(end 124.6 83.55)
 		(width 0.25)
 		(layer "B.Cu")
@@
 	)
 	(segment
-		(start 127.287199 88.885498)
-		(end 127.287199 94.5708)
+		(start 127.5 82.8)
+		(end 125.35 82.8)
 		(width 0.25)
 		(layer "B.Cu")
@@
 	)
 	(segment
-		(start 127.3 83)
-		(end 125.638299 83)
+		(start 124.6 87.171701)
+		(end 125.328299 87.9)
 		(width 0.25)
 		(layer "B.Cu")
@@
 	)
 	(segment
-		(start 124.885 83.753299)
-		(end 124.885 87.456701)
+		(start 127.325 88.125)
+		(end 127.325 94.532999)
 		(width 0.25)
 		(layer "B.Cu")
@@
 	)
 	(segment
-		(start 125.638299 83)
-		(end 124.885 83.753299)
+		(start 124.6 83.55)
+		(end 124.6 87.171701)
 		(width 0.25)
 		(layer "B.Cu")
@@
 	)
 	(segment
-		(start 125.528299 88.1)
-		(end 126.501701 88.1)
+		(start 125.328299 87.9)
+		(end 127.1 87.9)
 		(width 0.25)
 		(layer "B.Cu")
@@
 	)
 	(segment
-		(start 124.885 87.456701)
-		(end 125.528299 88.1)
+		(start 128.6 81.7)
+		(end 127.5 82.8)
 		(width 0.25)
 		(layer "B.Cu")
