File: expander_usb_sd/expander_usb_sd.kicad_sch (KiCad schematic)
At the start: 8 parts, among them J1 Micro_SD_Card_Det1, J2 USB power - Teensy device, J3 Internal_USB_Host_Teensy, J4 USB power - host

Commit message: most of USB+SD card expander done
Parts:
- removed External_USB_C_Teensy: USB_C_Plug_USB2.0, symbol Connector:USB_C_Plug_USB2.0
- removed Internal_USB_A_Teensy: USB_A, symbol Connector:USB_A
- added H1, H2: MountingHole, MountingHole:MountingHole_3.2mm_M3, symbol Mechanical:MountingHole
- added J5-TeensyMicroUSB1: USB 5 pin to Teensy/MicroUSB, Connector_PinHeader_2.54mm:PinHeader_1x05_P2.54mm_Vertical, symbol Connector:Conn_01x05_Pin
- added J6-USBHost1: USB 5 pin to frontpanel/Type C, Connector_PinHeader_2.54mm:PinHeader_1x05_P2.54mm_Vertical, symbol Connector:Conn_01x05_Pin
- External_USB_A_Host1: renamed from External_USB_A_Host; footprint (none) -> Connector_USB:USB_A_Molex_105057_Vertical
- J1: footprint (none) -> footprints:PJS008U-3000-0
- J1-TeensyPower1: renamed from J2; footprint (none) -> Connector_PinHeader_2.54mm:PinHeader_1x02_P2.54mm_Vertical
- J2: renamed from J3; footprint (none) -> Connector_PinHeader_2.54mm:PinHeader_1x05_P2.54mm_Vertical
- J2-USBHostPower1: renamed from J4; footprint (none) -> Connector_PinHeader_2.54mm:PinHeader_1x02_P2.54mm_Vertical
- SD_connector1: renamed from SD_connector; footprint (none) -> Connector_PinHeader_2.54mm:PinHeader_2x04_P2.54mm_Vertical
Connections:
- net GND: now also External_USB_A_Host1.5 (Shield), J1.10 (SHIELD), J2.5 (Pin_5)
- net at J1-TeensyPower1.2 (Pin_2): now also J6-USBHost1.1 (Pin_1)
- net at J2-USBHostPower1.1 (Pin_1): now also J2.1 (Pin_1)
- net at J2-USBHostPower1.2 (Pin_2): now also External_USB_A_Host1.1 (VBUS)
- net at J2.2 (Pin_2): now also External_USB_A_Host1.2 (D-)
- net at J2.3 (Pin_3): now also External_USB_A_Host1.3 (D+)
- net at J2.4 (Pin_4): now also External_USB_A_Host1.4 (GND)
Other:
- moved on the sheet: J1-TeensyPower1, J2

Commit message: updated to correct(?) footprint + 3d model for the usb socket
Parts:
- External_USB_A_Host1: footprint Connector_USB:USB_A_Molex_105057_Vertical -> USB-A1VSB6:ONSHORE_USB-A1VSB6; symbol Connector:USB_A -> USB-A1VSB6:USB-A1VSB6; MANUFACTURER (none) -> On Shore Technology; PARTREV (none) -> D; STANDARD (none) -> Manufacturer Recommendation
Connections:
- net GND: no longer External_USB_A_Host1.5 (Shield), J2.5 (Pin_5)
- net at External_USB_A_Host1.4 (GND), J2.4 (Pin_4): now also External_USB_A_Host1.S1 (SHIELD), External_USB_A_Host1.S2 (SHIELD__1), J2.5 (Pin_5)
Changed lines of the file:
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@@
 (kicad_sch (version 20230121) (generator eeschema)
   (paper "A4")
+  (junction (at 228.473 118.872) (diameter 0) (color 0 0 0 0)
+  )
+  (junction (at 228.473 121.412) (diameter 0) (color 0 0 0 0)
+  )
   (junction (at 70.104 138.938) (diameter 0) (color 0 0 0 0)
   )
   (junction (at 70.104 141.478) (diameter 0) (color 0 0 0 0)
   )
-  (junction (at 220.345 127.762) (diameter 0) (color 0 0 0 0)
+  (junction (at 209.804 123.952) (diameter 0) (color 0 0 0 0)
   )
   (junction (at 70.104 144.018) (diameter 0) (color 0 0 0 0)
@@
     (stroke (width 0) (type default))
   )
-  (wire (pts (xy 219.075 126.492) (xy 201.93 126.492))
+  (wire (pts (xy 209.804 116.332) (xy 228.473 116.332))
     (stroke (width 0) (type default))
   )
@@
     (stroke (width 0) (type default))
   )
+  (wire (pts (xy 209.804 113.792) (xy 228.473 113.792))
+    (stroke (width 0) (type default))
+  )
   (wire (pts (xy 75.565 57.658) (xy 67.945 57.658))
     (stroke (width 0) (type default))
@@
     (stroke (width 0) (type default))
   )
-  (wire (pts (xy 209.55 116.332) (xy 228.473 116.332))
-    (stroke (width 0) (type default))
-  )
-  (wire (pts (xy 217.043 113.792) (xy 217.043 118.872))
-    (stroke (width 0) (type default))
-  )
   (wire (pts (xy 67.945 65.278) (xy 83.439 65.278))
     (stroke (width 0) (type default))
@@
     (stroke (width 0) (type default))
   )
+  (wire (pts (xy 228.473 118.872) (xy 228.473 121.412))
+    (stroke (width 0) (type default))
+  )
   (wire (pts (xy 87.884 59.309) (xy 96.012 59.309))
     (stroke (width 0) (type default))
   )
-  (wire (pts (xy 199.39 127.762) (xy 199.39 126.492))
-    (stroke (width 0) (type default))
-  )
-  (wire (pts (xy 209.55 111.252) (xy 217.297 111.252))
+  (wire (pts (xy 209.804 118.872) (xy 228.473 118.872))
+    (stroke (width 0) (type default))
+  )
+  (wire (pts (xy 228.473 121.412) (xy 222.377 121.412))
     (stroke (width 0) (type default))
   )
@@
     (stroke (width 0) (type default))
   )
-  (wire (pts (xy 220.345 121.412) (xy 220.345 127.762))
+  (wire (pts (xy 209.804 123.952) (xy 209.804 126.492))
     (stroke (width 0) (type default))
   )
@@
     (stroke (width 0) (type default))
   )
-  (wire (pts (xy 228.473 118.872) (xy 219.075 118.872))
-    (stroke (width 0) (type default))
-  )
-  (wire (pts (xy 228.473 121.412) (xy 220.345 121.412))
+  (wire (pts (xy 209.804 123.444) (xy 209.804 123.952))
     (stroke (width 0) (type default))
   )
@@
     (stroke (width 0) (type default))
   )
-  (wire (pts (xy 228.473 113.792) (xy 217.043 113.792))
-    (stroke (width 0) (type default))
-  )
   (wire (pts (xy 67.945 60.198) (xy 89.916 60.198))
     (stroke (width 0) (type default))
@@
     (stroke (width 0) (type default))
   )
-  (wire (pts (xy 219.075 118.872) (xy 219.075 126.492))
-    (stroke (width 0) (type default))
-  )
-  (wire (pts (xy 220.345 127.762) (xy 199.39 127.762))
-    (stroke (width 0) (type default))
-  )
   (wire (pts (xy 69.977 144.018) (xy 70.104 144.018))
     (stroke (width 0) (type default))
@@
     (stroke (width 0) (type default))
   )
+  (wire (pts (xy 209.804 111.252) (xy 217.297 111.252))
+    (stroke (width 0) (type default))
+  )
+  (wire (pts (xy 209.804 123.444) (xy 222.377 123.444))
+    (stroke (width 0) (type default))
+  )
   (wire (pts (xy 69.977 138.938) (xy 70.104 138.938))
     (stroke (width 0) (type default))
@@
     (stroke (width 0) (type default))
   )
-  (wire (pts (xy 217.043 118.872) (xy 209.55 118.872))
+  (wire (pts (xy 222.377 121.412) (xy 222.377 123.444))
     (stroke (width 0) (type default))
   )
@@
     )
   )
-  (symbol (lib_id "PCM_4ms_Power-symbol:GND") (at 220.345 127.762 0) (unit 1)
-    (in_bom yes) (on_board yes) (dnp no) (fields_autoplaced)
-    (property "Reference" "#PWR02" (at 220.345 134.112 0)
-      (effects (font (size 1.27 1.27)) hide)
-    )
-    (property "Value" "GND" (at 220.345 131.8975 0)
-      (effects (font (size 1.27 1.27)))
-    )
-    (property "Footprint" "" (at 220.345 127.762 0)
-      (effects (font (size 1.27 1.27)) hide)
-    )
-    (property "Datasheet" "" (at 220.345 127.762 0)
-      (effects (font (size 1.27 1.27)) hide)
-    )
-    (pin "1")
-    (instances
-      (project "expander_usb_sd"
-        (path "/a9e4ad89-ca26-464a-b121-56ca282a5e7f"
-          (reference "#PWR02") (unit 1)
-        )
-      )
-    )
-  )
   (symbol (lib_id "Mechanical:MountingHole") (at 262.382 110.871 0) (unit 1)
     (in_bom yes) (on_board yes) (dnp no) (fields_autoplaced)
@@
     )
   )
-  (symbol (lib_id "Connector:USB_A") (at 201.93 116.332 0) (unit 1)
-    (in_bom yes) (on_board yes) (dnp no)
-    (property "Reference" "External_USB_A_Host1" (at 192.151 117.602 90)
-      (effects (font (size 1.27 1.27)))
-    )
-    (property "Value" "USB_A" (at 201.93 107.6231 0)
-      (effects (font (size 1.27 1.27)))
-    )
-    (property "Footprint" "Connector_USB:USB_A_Molex_105057_Vertical" (at 205.74 117.602 0)
-      (effects (font (size 1.27 1.27)) hide)
-    )
-    (property "Datasheet" " ~" (at 205.74 117.602 0)
-      (effects (font (size 1.27 1.27)) hide)
+  (symbol (lib_id "USB-A1VSB6:USB-A1VSB6") (at 199.644 116.332 0) (mirror y) (unit 1)
+    (in_bom yes) (on_board yes) (dnp no)
+    (property "Reference" "External_USB_A_Host1" (at 199.263 135.255 0)
+      (effects (font (size 1.27 1.27)))
+    )
+    (property "Value" "USB_A" (at 199.644 107.6231 0)
+      (effects (font (size 1.27 1.27)))
+    )
+    (property "Footprint" "USB-A1VSB6:ONSHORE_USB-A1VSB6" (at 199.644 116.332 0)
+      (effects (font (size 1.27 1.27)) (justify bottom) hide)
+    )
+    (property "Datasheet" " ~" (at 199.644 116.332 0)
+      (effects (font (size 1.27 1.27)) hide)
+    )
+    (property "PARTREV" "D" (at 199.644 116.332 0)
+      (effects (font (size 1.27 1.27)) (justify bottom) hide)
+    )
+    (property "STANDARD" "Manufacturer Recommendation" (at 199.644 116.332 0)
+      (effects (font (size 1.27 1.27)) (justify bottom) hide)
+    )
+    (property "MANUFACTURER" "On Shore Technology" (at 199.644 116.332 0)
+      (effects (font (size 1.27 1.27)) (justify bottom) hide)
     )
     (pin "1")
@@
     (pin "3")
     (pin "4")
-    (pin "5")
-    (instances
-      (project "expander_usb_sd"
+    (pin "S1")
+    (pin "S2")
+    (instances
+      (project "expander_usb_sd"

Commit message: fucking connect the USB Host pins that were completely unconnected previously... facepalm!
Connections:
- net at J1-TeensyPower1.1 (Pin_1): now also J5-TeensyMicroUSB1.1 (Pin_1)
- net at J6-USBHost1.2 (Pin_2): now also J5-TeensyMicroUSB1.2 (Pin_2)
- net at J6-USBHost1.3 (Pin_3): now also J5-TeensyMicroUSB1.3 (Pin_3)
- net at J6-USBHost1.4 (Pin_4): now also J5-TeensyMicroUSB1.4 (Pin_4)
- net at J6-USBHost1.5 (Pin_5): now also J5-TeensyMicroUSB1.5 (Pin_5)
Changed lines of the file:
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@@
   (junction (at 228.473 121.412) (diameter 0) (color 0 0 0 0)
   )
-  (junction (at 70.104 138.938) (diameter 0) (color 0 0 0 0)
-  )
-  (junction (at 70.104 141.478) (diameter 0) (color 0 0 0 0)
-  )
   (junction (at 209.804 123.952) (diameter 0) (color 0 0 0 0)
   )
-  (junction (at 70.104 144.018) (diameter 0) (color 0 0 0 0)
-  )
-  (junction (at 70.104 149.098) (diameter 0) (color 0 0 0 0)
-  )
-  (junction (at 70.104 146.558) (diameter 0) (color 0 0 0 0)
-  )
   (wire (pts (xy 96.012 66.929) (xy 75.565 66.929))
     (stroke (width 0) (type default))
   )
-  (wire (pts (xy 69.977 149.098) (xy 70.104 149.098))
+  (wire (pts (xy 69.977 149.098) (xy 91.059 149.098))
     (stroke (width 0) (type default))
   )
@@
     (stroke (width 0) (type default))
   )
-  (wire (pts (xy 69.977 141.478) (xy 70.104 141.478))
+  (wire (pts (xy 69.977 141.478) (xy 91.059 141.478))
     (stroke (width 0) (type default))
   )
@@
     (stroke (width 0) (type default))
   )
-  (wire (pts (xy 70.104 141.478) (xy 91.059 141.478))
-    (stroke (width 0) (type default))
-  )
   (wire (pts (xy 228.473 118.872) (xy 228.473 121.412))
     (stroke (width 0) (type default))
@@
     (stroke (width 0) (type default))
   )
-  (wire (pts (xy 70.104 146.558) (xy 91.059 146.558))
-    (stroke (width 0) (type default))
-  )
   (wire (pts (xy 43.053 57.658) (xy 43.053 69.469))
     (stroke (width 0) (type default))
@@
     (stroke (width 0) (type default))
   )
-  (wire (pts (xy 69.977 146.558) (xy 70.104 146.558))
+  (wire (pts (xy 69.977 146.558) (xy 91.059 146.558))
     (stroke (width 0) (type default))
   )
@@
     (stroke (width 0) (type default))
   )
-  (wire (pts (xy 70.104 138.938) (xy 79.502 138.938))
-    (stroke (width 0) (type default))
-  )
   (wire (pts (xy 67.945 60.198) (xy 89.916 60.198))
     (stroke (width 0) (type default))
@@
     (stroke (width 0) (type default))
   )
-  (wire (pts (xy 70.104 149.098) (xy 91.059 149.098))
-    (stroke (width 0) (type default))
-  )
-  (wire (pts (xy 69.977 144.018) (xy 70.104 144.018))
+  (wire (pts (xy 69.977 144.018) (xy 91.059 144.018))
     (stroke (width 0) (type default))
   )
@@
     (stroke (width 0) (type default))
   )
-  (wire (pts (xy 70.104 144.018) (xy 91.059 144.018))
-    (stroke (width 0) (type default))
-  )
   (wire (pts (xy 209.804 111.252) (xy 217.297 111.252))
     (stroke (width 0) (type default))
@@
     (stroke (width 0) (type default))
   )
-  (wire (pts (xy 69.977 138.938) (xy 70.104 138.938))
+  (wire (pts (xy 69.977 138.938) (xy 79.502 138.938))
     (stroke (width 0) (type default))
   )
@@
     )
   )
-  (symbol (lib_id "Connector:Conn_01x05_Pin") (at 65.024 144.018 0) (unit 1)
-    (in_bom yes) (on_board yes) (dnp no)
-    (property "Reference" "J6-USBHost1" (at 61.341 139.7 90)
+  (symbol (lib_id "Connector:Conn_01x05_Pin") (at 64.897 144.018 0) (unit 1)
+    (in_bom yes) (on_board yes) (dnp no)
+    (property "Reference" "J6-USBHost1" (at 61.214 139.7 90)
       (effects (font (size 1.27 1.27)) (justify right))
     )
-    (property "Value" "USB 5 pin to frontpanel/Type C" (at 57.277 128.524 90)
+    (property "Value" "USB 5 pin to frontpanel/Type C" (at 57.15 128.524 90)
       (effects (font (size 1.27 1.27)) (justify right))
     )
-    (property "Footprint" "Connector_PinHeader_2.54mm:PinHeader_1x05_P2.54mm_Vertical" (at 65.024 144.018 0)
-      (effects (font (size 1.27 1.27)) hide)
-    )
-    (property "Datasheet" "~" (at 65.024 144.018 0)
+    (property "Footprint" "Connector_PinHeader_2.54mm:PinHeader_1x05_P2.54mm_Vertical" (at 64.897 144.018 0)
+      (effects (font (size 1.27 1.27)) hide)
+    )
+    (property "Datasheet" "~" (at 64.897 144.018 0)
       (effects (font (size 1.27 1.27)) hide)
     )
@@
     )
   )
-  (symbol (lib_id "Connector:Conn_01x05_Pin") (at 96.266 144.018 0) (mirror y) (unit 1)
-    (in_bom yes) (on_board yes) (dnp no)
-    (property "Reference" "J5-TeensyMicroUSB1" (at 99.568 143.764 90)
-      (effects (font (size 1.27 1.27)))
-    )
-    (property "Value" "USB 5 pin to Teensy/MicroUSB" (at 103.886 143.002 90)
-      (effects (font (size 1.27 1.27)))
-    )
-    (property "Footprint" "Connector_PinHeader_2.54mm:PinHeader_1x05_P2.54mm_Vertical" (at 96.266 144.018 0)
-      (effects (font (size 1.27 1.27)) hide)
-    )
-    (property "Datasheet" "~" (at 96.266 144.018 0)
-      (effects (font (size 1.27 1.27)) hide)
-    )
+  (symbol (lib_id "Connector:Conn_01x05_Pin") (at 96.139 144.018 0) (mirror y) (unit 1)
+    (in_bom yes) (on_board yes) (dnp no)
+    (property "Reference" "J5-TeensyMicroUSB1" (at 99.441 143.764 90)
+      (effects (font (size 1.27 1.27)))
+    )
+    (property "Value" "USB 5 pin to Teensy/MicroUSB" (at 103.759 143.002 90)
+      (effects (font (size 1.27 1.27)))
+    )
+    (property "Footprint" "Connector_PinHeader_2.54mm:PinHeader_1x05_P2.54mm_Vertical" (at 96.139 144.018 0)
+      (effects (font (size 1.27 1.27)) hide)
+    )
+    (property "Datasheet" "~" (at 96.139 144.018 0)
+      (effects (font (size 1.27 1.27)) hide)
+    )

Commit message: fixed yet more dumb routing errors on the usb_sd; probably still isn't ready to use
Parts:
- renumbered J2-USBHostPower1 to USBHostPower1
Connections:
- net GND: now also External_USB_A_Host1.4 (GND)
- net at External_USB_A_Host1.S1 (SHIELD), External_USB_A_Host1.S2 (SHIELD__1), J2.4 (Pin_4)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: no longer External_USB_A_Host1.4 (GND)
Other:
- moved on the sheet: External_USB_A_Host1, J2, USBHostPower1

Commit message: believe fixed problems with expander_usb_sd; tracked a bunch of stuff that was untracked (expander_cv_output?)
Connections:
- net GND: no longer External_USB_A_Host1.4 (GND)
- net at External_USB_A_Host1.S1 (SHIELD), External_USB_A_Host1.S2 (SHIELD__1), J2.4 (Pin_4)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: now also External_USB_A_Host1.4 (GND)
Changed lines of the file:
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@@
+	)
+	(junction
+		(at 209.55 121.92)
+		(diameter 0)
+		(color 0 0 0 0)
 	)
 	(junction
@@
 	(wire
 		(pts
-			(xy 217.17 111.76) (xy 209.55 111.76)
-		)
-		(stroke
-			(width 0)
-			(type default)
-		)
-	)
-	(wire
-		(pts
 			(xy 85.471 62.738) (xy 85.471 56.769)
 		)
@@
 	(wire
 		(pts
+			(xy 209.55 111.76) (xy 217.17 111.76)
+		)
+		(stroke
+			(width 0)
+			(type default)
+		)
+	)
+	(wire
+		(pts
 			(xy 46.99 62.738) (xy 46.99 68.326)
 		)
@@
 		(pts
 			(xy 85.471 56.769) (xy 96.012 56.769)
+		)
+		(stroke
+			(width 0)
+			(type default)
+		)
+	)
+	(wire
+		(pts
+			(xy 209.55 119.38) (xy 209.55 121.92)
 		)
 		(stroke
@@
 					(unit 1)
 				)
-			)
-		)
-	)
-	(symbol
-		(lib_id "PCM_4ms_Power-symbol:GND")
-		(at 209.55 119.38 90)
-		(unit 1)
-		(exclude_from_sim no)
-		(in_bom yes)
-		(on_board yes)
-		(dnp no)
-		(fields_autoplaced yes)
-		(property "Reference" "#PWR02"
-			(at 215.9 119.38 0)
-			(effects
-				(font
-					(size 1.27 1.27)
-				)
-				(hide yes)
-			)
-		)
-		(property "Value" "GND"
-			(at 212.725 119.6968 90)
-			(effects
-				(font
-					(size 1.27 1.27)
-				)
-				(justify right)
-			)
-		)
-		(property "Footprint" ""
-			(at 209.55 119.38 0)
-			(effects
-				(font
-					(size 1.27 1.27)
-				)
-				(hide yes)
-			)
-		)
-		(property "Datasheet" ""
-			(at 209.55 119.38 0)
-			(effects
-				(font
-					(size 1.27 1.27)
-				)
-				(hide yes)
-			)
-		)
-		(property "Description" ""
-			(at 209.55 119.38 0)
-			(effects
-				(font
-					(size 1.27 1.27)
-				)
-				(hide yes)
-			)
-		)
-		(pin "1"
-		)
-		(instances
-			(project "expander_usb_sd"
-				(path "/a9e4ad89-ca26-464a-b121-56ca282a5e7f"
-					(reference "#PWR02")
-					(unit 1)
-				)
