File: expander_cv_output/expander_cv_output/dac2.kicad_sch (KiCad schematic)
At the start: 32 parts, among them U1 TL074, U2 TL074, U6 MCP4728

Commit message: tracked first draft of expander_cv_output
Parts:
- removed C4: C_Small, Capacitor_SMD:C_0805_2012Metric_Pad1.18x1.45mm_HandSolder, symbol Device:C_Small
- removed D10, D7, D8, D9: LED_Dual_Bidirectional, LED_THT:LED_D3.0mm, symbol Device:LED_Dual_Bidirectional
- removed R21, R22, R23, R24, R31, R32, R33, R34: 100K, Resistor_SMD:R_0603_1608Metric_Pad0.98x0.95mm_HandSolder, symbol Device:R
- removed R25, R26, R35, R36: 56K, Resistor_SMD:R_0603_1608Metric_Pad0.98x0.95mm_HandSolder, symbol Device:R
- removed R27, R28, R37, R38: 470k, Resistor_SMD:R_0603_1608Metric_Pad0.98x0.95mm_HandSolder, symbol Device:R
- removed R29, R30, R39, R40: 1K, Resistor_SMD:R_0603_1608Metric_Pad0.98x0.95mm_HandSolder, symbol Device:R
- removed RV5, RV6, RV7, RV8: R_Potentiometer_Small, Potentiometer_THT:Potentiometer_Bourns_3296X_Horizontal, symbol Device:R_Potentiometer_Small
- removed U1, U2: TL074, Package_SO:TSSOP-14_4.4x5mm_P0.65mm, symbol Amplifier_Operational:TL074
- removed U6: MCP4728, Package_SO:MSOP-10_3x3mm_P0.5mm, symbol Analog_DAC:MCP4728
