File: expander_cv_output/expander_cv_output/expander_cv_output.kicad_sch (KiCad schematic)
At the start: 22 parts, among them J1 Conn_01x10_Pin, J2 Conn_01x10_Socket, J3 Conn_01x08_Pin, J4 Conn_01x08_Socket, J5 Conn_01x08_Socket, J6 Conn_01x08_Pin, U1 TL074, U2 TL074

Commit message: tracked first draft of expander_cv_output
Parts:
- removed CV_INPUT_I2C_EXPANDER_MAIN1: 8 pin header, Connector_PinHeader_2.54mm:PinHeader_2x04_P2.54mm_Vertical, symbol Connector_Generic:Conn_02x04_Odd_Even
- removed J1: Conn_01x10_Pin, Connector_PinHeader_2.54mm:PinHeader_1x10_P2.54mm_Vertical, symbol Connector:Conn_01x10_Pin
- removed J2: Conn_01x10_Socket, Connector_PinSocket_2.54mm:PinSocket_1x10_P2.54mm_Vertical, symbol Connector:Conn_01x10_Socket
- removed J3, J6: Conn_01x08_Pin, Connector_PinSocket_2.54mm:PinSocket_1x08_P2.54mm_Vertical, symbol Connector:Conn_01x08_Pin
- removed J4, J5: Conn_01x08_Socket, Connector_PinSocket_2.54mm:PinSocket_1x08_P2.54mm_Vertical, symbol Connector:Conn_01x08_Socket
- removed JACK1, JACK2, JACK3, JACK4, JACK5, JACK6, JACK7, JACK8: AudioJack2_SwitchT, Connector_Audio:Jack_3.5mm_QingPu_WQP-PJ398SM_Vertical_CircularHoles, symbol Connector_Audio:AudioJack2_SwitchT
- added ADDR_A0, ADDR_A1, ADDR_A2, ADDR_A3: Conn_01x03_Pin, Jumper:SolderJumper-3_P1.3mm_Open_RoundedPad1.0x1.5mm, symbol Connector:Conn_01x03_Pin
- added C1, C19, C2, C5, C6, C7, C9: 100nF, Capacitor_SMD:C_0805_2012Metric_Pad1.18x1.45mm_HandSolder, symbol Device:C_Small
- added C8: 10uF, Capacitor_SMD:C_0805_2012Metric_Pad1.18x1.45mm_HandSolder, symbol Device:C_Small
- added DAC1: DAC8574IPWG4, Package_SO:TSSOP-16_4.4x5mm_P0.65mm, symbol dac8754:DAC8574IPWG4
- added J1: Future?, Connector_PinHeader_2.54mm:PinHeader_1x02_P2.54mm_Vertical, symbol Connector:Conn_01x02_Pin
- added J2, J7: Conn_02x05_Odd_Even, Connector_IDC:IDC-Header_2x05_P2.54mm_Vertical, symbol Connector_Generic:Conn_02x05_Odd_Even
- added J3: SDA pullup, Connector_PinHeader_2.54mm:PinHeader_1x02_P2.54mm_Vertical, symbol Connector:Conn_01x02_Pin
- added J4: SCL pullup, Connector_PinHeader_2.54mm:PinHeader_1x02_P2.54mm_Vertical, symbol Connector:Conn_01x02_Pin
- added JACK_A1, JACK_B1, JACK_C1, JACK_D1: PJ302M, Kicad_Akiyuki_Footprint:PJ302M, symbol Akiyuki_Connector:PJ302M
- added R1, R5, R6: 10k, Resistor_SMD:R_0805_2012Metric_Pad1.20x1.40mm_HandSolder, symbol Device:R
- added R2: 560, Resistor_SMD:R_0805_2012Metric_Pad1.20x1.40mm_HandSolder, symbol Device:R
- added R3, R4: 150r, Resistor_SMD:R_0805_2012Metric_Pad1.20x1.40mm_HandSolder, symbol Device:R
- added U3: LM4040DBZ-5, Package_TO_SOT_SMD:SOT-23_Handsoldering, symbol Reference_Voltage:LM4040DBZ-5
- added U4: LD1117S33TR_SOT223, Package_TO_SOT_SMD:SOT-223, symbol Regulator_Linear:LD1117S33TR_SOT223
- added U5: LM4040DBZ-33, Package_TO_SOT_SMD:SOT-23_Handsoldering, symbol Reference_Voltage:LM4040DBZ-5
- C3: renamed from C1; value C_Polarized_Small -> 10uF; footprint Capacitor_THT:CP_Radial_D5.0mm_P2.50mm -> Capacitor_SMD:CP_Elec_5x5.7
- C4: renamed from C2; value C_Polarized_Small -> 10uF; footprint Capacitor_THT:CP_Radial_D5.0mm_P2.50mm -> Capacitor_SMD:CP_Elec_5x5.7
- D1, D2: value D_Small -> 1N5817
- U1, U2: footprint Package_SO:TSSOP-14_4.4x5mm_P0.65mm -> Package_SO:SOIC-14_3.9x8.7mm_P1.27mm
Connections:
- net +5V from Host: now also J2.6 (Pin_6), J2.8 (Pin_8), J7.6 (Pin_6), J7.8 (Pin_8)
- net -12V: now also C5.2, C6.1
- net 12V: now also C1.1, C2.1, R1.1, R2.1
- net 5V: now also ADDR_A0.3 (Pin_3), ADDR_A1.3 (Pin_3), ADDR_A2.3 (Pin_3), ADDR_A3.3 (Pin_3), C7.2, C9.2, DAC1.4 (VDD), U4.3 (VI)
- net GND: now also ADDR_A0.1 (Pin_1), ADDR_A1.1 (Pin_1), ADDR_A2.1 (Pin_1), ADDR_A3.1 (Pin_1), C1.2, C19.1, C2.2, C5.1, C6.2, C7.1, C8.1, C9.1, DAC1.5 (VREFL), DAC1.6 (GND), DAC1.9 (LDAC), J2.2 (Pin_2), J2.4 (Pin_4), J7.2 (Pin_2), J7.4 (Pin_4), JACK_A1.1, JACK_B1.1, JACK_C1.1, JACK_D1.1, R4.2, U3.2 (A), U4.1 (GND), U5.2 (A)
- net Output Backboard A: now also JACK_A1.3
- net Output Backboard B: now also JACK_B1.3
- net Output Backboard C: now also JACK_C1.3
- net Output Backboard D: now also JACK_D1.3
- net i2c SCL: now also DAC1.10 (SCL), J2.1 (Pin_1), J2.5 (Pin_5), J7.1 (Pin_1), J7.5 (Pin_5), R6.2
- net i2c SDA: now also DAC1.11 (SDA), J2.3 (Pin_3), J2.7 (Pin_7), J7.3 (Pin_3), J7.7 (Pin_7), R5.2
- new net: J1.1 (Pin_1), J2.10 (Pin_10), J7.10 (Pin_10)
- new net: J1.2 (Pin_2), J2.9 (Pin_9), J7.9 (Pin_9)
- new net: J3.2 (Pin_2), R5.1
- new net: J4.2 (Pin_2), R6.1
- new net: ADDR_A3.2 (Pin_2), DAC1.16 (A3)
- new net: ADDR_A2.2 (Pin_2), DAC1.15 (A2)
- new net: ADDR_A0.2 (Pin_2), DAC1.13 (A0)
- new net: ADDR_A1.2 (Pin_2), DAC1.14 (A1)
- new net 1.65v reference: R3.2, R4.1
- new net 3.3V: C19.2, C8.2, DAC1.12 (IOVDD), J3.1 (Pin_1), J4.1 (Pin_1), U4.2 (VO)
- new net 3.3v reference: R2.2, R3.1, U5.1 (K)
- new net 5v reference: DAC1.3 (VREFH), R1.2, U3.1 (K)
- new net DAC output 1: DAC1.1 (VOUTA)
- new net DAC output 2: DAC1.2 (VOUTB)
- new net DAC output 3: DAC1.7 (VOUTC)
- new net DAC output 4: DAC1.8 (VOUTD)
- new net Normal A: JACK_A1.2
- new net Normal B: JACK_B1.2
- new net Normal C: JACK_C1.2
Other:
- removed sheet DAC 2
- added sheet CV input (cv_input.kicad_sch)
- moved on the sheet: C3, C4, D1, D2
