File: expander_cv_output/expander_cv_output/expander_cv_output.kicad_pcb (KiCad board)
At the start: 2 copper layers, 112.5 x 128.5 mm, 84 parts, among them J1 Conn_01x10_Pin, J2 Conn_01x10_Socket, J3 Conn_01x08_Pin, J4 Conn_01x08_Socket, J5 Conn_01x08_Socket, J6 Conn_01x08_Pin, U1 TL074, U2 TL074, U3 TL074, U4 MCP4728, U5 TL074, U6 MCP4728

Commit message: tracked first draft of expander_cv_output
Parts:
- removed CV_INPUT_I2C_EXPANDER_MAIN1: 8 pin header, Connector_PinHeader_2.54mm:PinHeader_2x04_P2.54mm_Vertical
- removed D10, D3, D4, D5, D6, D7, D8, D9: LED_Dual_Bidirectional, LED_THT:LED_D3.0mm
- removed J1: Conn_01x10_Pin, Connector_PinHeader_2.54mm:PinHeader_1x10_P2.54mm_Vertical
- removed J6: Conn_01x08_Pin, Connector_PinSocket_2.54mm:PinSocket_1x08_P2.54mm_Vertical
- removed JACK1, JACK2, JACK3, JACK4, JACK5, JACK6, JACK7, JACK8: AudioJack2_SwitchT, Connector_Audio:Jack_3.5mm_QingPu_WQP-PJ398SM_Vertical_CircularHoles
- removed R27, R28, R37, R38: 470k, Resistor_SMD:R_0603_1608Metric_Pad0.98x0.95mm_HandSolder
- removed R29, R30, R39, R40: 1K, Resistor_SMD:R_0603_1608Metric_Pad0.98x0.95mm_HandSolder
- removed R31, R32, R33, R34: 100K, Resistor_SMD:R_0603_1608Metric_Pad0.98x0.95mm_HandSolder
- removed R35, R36: 56K, Resistor_SMD:R_0603_1608Metric_Pad0.98x0.95mm_HandSolder
- removed RV1, RV2, RV3, RV4, RV5, RV6, RV7, RV8: R_Potentiometer_Small, Potentiometer_THT:Potentiometer_Bourns_3296X_Horizontal
- removed U6: MCP4728, Package_SO:MSOP-10_3x3mm_P0.5mm
- added ADDR_A0: Conn_01x03_Pin, Jumper:SolderJumper-3_P1.3mm_Open_RoundedPad1.0x1.5mm, B.Cu at (162.6, 94.9)
- added ADDR_A1: Conn_01x03_Pin, Jumper:SolderJumper-3_P1.3mm_Open_RoundedPad1.0x1.5mm, B.Cu at (162.6, 91.1)
- added ADDR_A2: Conn_01x03_Pin, Jumper:SolderJumper-3_P1.3mm_Open_RoundedPad1.0x1.5mm, B.Cu at (162.6, 87.1)
- added ADDR_A3: Conn_01x03_Pin, Jumper:SolderJumper-3_P1.3mm_Open_RoundedPad1.0x1.5mm, B.Cu at (162.6, 83.4)
- added ADS1015_2_DIG1: ADS1015 digital side, Connector_PinSocket_2.54mm:PinSocket_1x05_P2.54mm_Vertical, F.Cu at (132.1, 101.6)
- added ASD1015_2_ANA1: ADS1015 analog side, Connector_PinSocket_2.54mm:PinSocket_1x05_P2.54mm_Vertical, F.Cu at (149.9, 101.6)
- added C10: 22pF, Capacitor_SMD:C_0805_2012Metric_Pad1.18x1.45mm_HandSolder, F.Cu at (146.7, 32.4)
- added C11: 22pF, Capacitor_SMD:C_0805_2012Metric_Pad1.18x1.45mm_HandSolder, F.Cu at (144.9, 51.0)
- added C12: 100nF, Capacitor_SMD:C_0805_2012Metric_Pad1.18x1.45mm_HandSolder, F.Cu at (148.9, 36.6)
- added C13: 100nF, Capacitor_SMD:C_0805_2012Metric_Pad1.18x1.45mm_HandSolder, F.Cu at (151.0, 50.5)
- added C14: 22pF, Capacitor_SMD:C_0805_2012Metric_Pad1.18x1.45mm_HandSolder, F.Cu at (145.2, 77.2)
- added C15: 22pF, Capacitor_SMD:C_0805_2012Metric_Pad1.18x1.45mm_HandSolder, F.Cu at (144.5, 92.9)
- added C16: 100nF, Capacitor_SMD:C_0805_2012Metric_Pad1.18x1.45mm_HandSolder, F.Cu at (157.0, 58.7)
- added C17: 100nF, Capacitor_SMD:C_0805_2012Metric_Pad1.18x1.45mm_HandSolder, F.Cu at (157.1, 76.3)
- added C18: 100nF, Capacitor_SMD:C_0805_2012Metric_Pad1.18x1.45mm_HandSolder, F.Cu at (131.3, 96.2)
- added C19: 100nF, Capacitor_SMD:C_0805_2012Metric_Pad1.18x1.45mm_HandSolder, F.Cu at (152.1, 63.9)
- added C5: 100nF, Capacitor_SMD:C_0805_2012Metric_Pad1.18x1.45mm_HandSolder, F.Cu at (152.5, 42.4)
- added C6: 100nF, Capacitor_SMD:C_0805_2012Metric_Pad1.18x1.45mm_HandSolder, F.Cu at (152.2, 84.4)
- added C7: 100nF, Capacitor_SMD:C_0805_2012Metric_Pad1.18x1.45mm_HandSolder, F.Cu at (137.4, 102.6)
- added C8: 10uF, Capacitor_SMD:C_0805_2012Metric_Pad1.18x1.45mm_HandSolder, F.Cu at (141.3, 102.6)
- added C9: 100nF, Capacitor_SMD:C_0805_2012Metric_Pad1.18x1.45mm_HandSolder, F.Cu at (147.5, 95.6)
- added DAC1: DAC8574IPWG4, Package_SO:TSSOP-16_4.4x5mm_P0.65mm, F.Cu at (147.1, 61.6)
- added J7: Conn_02x05_Odd_Even, Connector_IDC:IDC-Header_2x05_P2.54mm_Vertical, F.Cu at (136.2, 88.2)
- added JACK_A1: PJ302M, Kicad_Akiyuki_Footprint:PJ302M, F.Cu at (170.4, 34.6)
- added JACK_A2: PJ302M, Kicad_Akiyuki_Footprint:PJ302M, F.Cu at (170.4, 101.0)
- added JACK_B1: PJ302M, Kicad_Akiyuki_Footprint:PJ302M, F.Cu at (170.4, 52.0)
- added JACK_B2: PJ302M, Kicad_Akiyuki_Footprint:PJ302M, F.Cu at (170.4, 113.2)
- added JACK_C1: PJ302M, Kicad_Akiyuki_Footprint:PJ302M, F.Cu at (170.4, 69.4)
- added JACK_C2: PJ302M, Kicad_Akiyuki_Footprint:PJ302M, F.Cu at (170.4, 125.5)
- added JACK_D1: PJ302M, Kicad_Akiyuki_Footprint:PJ302M, F.Cu at (170.4, 86.8)
- added LED_A1: LED_Dual_Bidirectional, LED_THT:LED_D3.0mm, F.Cu at (162.6, 25.2)
- added LED_B1: LED_Dual_Bidirectional, LED_THT:LED_D3.0mm, F.Cu at (162.6, 42.6)
- added LED_C1: LED_Dual_Bidirectional, LED_THT:LED_D3.0mm, F.Cu at (162.5, 60.0)
- added LED_D1: LED_Dual_Bidirectional, LED_THT:LED_D3.0mm, F.Cu at (162.5, 77.4)
- C1, C2: value C_Polarized_Small -> 100nF; footprint Capacitor_THT:CP_Radial_D5.0mm_P2.50mm -> Capacitor_SMD:C_0805_2012Metric_Pad1.18x1.45mm_HandSolder
- C3, C4: value C_Small -> 10uF; footprint Capacitor_SMD:C_0805_2012Metric_Pad1.18x1.45mm_HandSolder -> Capacitor_SMD:CP_Elec_5x5.7
- D1, D2: value D_Small -> 1N5817
- EURO_POWER1: moved to F.Cu
- J2: value Conn_01x10_Socket -> Conn_02x05_Odd_Even; footprint Connector_PinSocket_2.54mm:PinSocket_1x10_P2.54mm_Vertical -> Connector_IDC:IDC-Header_2x05_P2.54mm_Vertical
- J3: value Conn_01x08_Pin -> SDA pullup; footprint Connector_PinSocket_2.54mm:PinSocket_1x08_P2.54mm_Vertical -> Connector_PinHeader_2.54mm:PinHeader_1x02_P2.54mm_Vertical; moved to F.Cu
- J4: value Conn_01x08_Socket -> SCL pullup; footprint Connector_PinSocket_2.54mm:PinSocket_1x08_P2.54mm_Vertical -> Connector_PinHeader_2.54mm:PinHeader_1x02_P2.54mm_Vertical
- J5: value Conn_01x08_Socket -> Conn_02x08_Counter_Clockwise; footprint Connector_PinSocket_2.54mm:PinSocket_1x08_P2.54mm_Vertical -> Connector_PinHeader_2.54mm:PinHeader_2x08_P2.54mm_Vertical
- R1: value 100K -> 10k; footprint Resistor_SMD:R_0603_1608Metric_Pad0.98x0.95mm_HandSolder -> Resistor_SMD:R_0805_2012Metric_Pad1.20x1.40mm_HandSolder
- R10, R19, R20, R9: value 1K -> 2.2k; footprint Resistor_SMD:R_0603_1608Metric_Pad0.98x0.95mm_HandSolder -> Resistor_SMD:R_0805_2012Metric_Pad1.20x1.40mm_HandSolder
- R11, R12, R21, R22: value 100K -> 220; footprint Resistor_SMD:R_0603_1608Metric_Pad0.98x0.95mm_HandSolder -> Resistor_SMD:R_0805_2012Metric_Pad1.20x1.40mm_HandSolder
- R13, R14, R23, R24: value 100K -> 1K; footprint Resistor_SMD:R_0603_1608Metric_Pad0.98x0.95mm_HandSolder -> Resistor_SMD:R_0805_2012Metric_Pad1.20x1.40mm_HandSolder
- R15, R16, R25, R26: value 56K -> 47; footprint Resistor_SMD:R_0603_1608Metric_Pad0.98x0.95mm_HandSolder -> Resistor_SMD:R_0805_2012Metric_Pad1.20x1.40mm_HandSolder
- R17, R18, R7, R8: value 470k -> 1K; footprint Resistor_SMD:R_0603_1608Metric_Pad0.98x0.95mm_HandSolder -> Resistor_SMD:R_0805_2012Metric_Pad1.20x1.40mm_HandSolder
- R2: value 100K -> 560; footprint Resistor_SMD:R_0603_1608Metric_Pad0.98x0.95mm_HandSolder -> Resistor_SMD:R_0805_2012Metric_Pad1.20x1.40mm_HandSolder
- R3, R4: value 100K -> 150r; footprint Resistor_SMD:R_0603_1608Metric_Pad0.98x0.95mm_HandSolder -> Resistor_SMD:R_0805_2012Metric_Pad1.20x1.40mm_HandSolder
- R5, R6: value 56K -> 10k; footprint Resistor_SMD:R_0603_1608Metric_Pad0.98x0.95mm_HandSolder -> Resistor_SMD:R_0805_2012Metric_Pad1.20x1.40mm_HandSolder
- U1, U2: footprint Package_SO:TSSOP-14_4.4x5mm_P0.65mm -> Package_SO:SOIC-14_3.9x8.7mm_P1.27mm
- U3: value TL074 -> LM4040DBZ-5; footprint Package_SO:TSSOP-14_4.4x5mm_P0.65mm -> Package_TO_SOT_SMD:SOT-23_Handsoldering
- U4: value MCP4728 -> LD1117S33TR_SOT223; footprint Package_SO:MSOP-10_3x3mm_P0.5mm -> Package_TO_SOT_SMD:SOT-223
- U5: value TL074 -> LM4040DBZ-33; footprint Package_SO:TSSOP-14_4.4x5mm_P0.65mm -> Package_TO_SOT_SMD:SOT-23_Handsoldering
- moved C1 83.3 mm to (142.1, 42.4), turned to 180 degrees
- moved U5 78.9 mm to (141.8, 106.8), turned to -90 degrees
- moved R13 72.0 mm to (167.9, 26.7), turned to -90 degrees
- moved U1 70.2 mm to (147.7, 43.6)
- moved U3 68.6 mm to (137.2, 106.8), turned to -90 degrees
- moved R11 64.8 mm to (151.0, 36.6), turned to -90 degrees
- moved J5 63.9 mm to (132.6, 48.9)
- moved R14 61.5 mm to (167.9, 44.1), turned to -90 degrees
- moved R25 60.2 mm to (157.0, 61.4)
- moved R20 56.5 mm to (144.4, 88.7), turned to 180 degrees
- moved R17 55.4 mm to (150.7, 76.0), turned to -90 degrees
- moved C4 51.9 mm to (134.9, 118.2)
- moved R12 50.7 mm to (148.3, 50.3), turned to -90 degrees
- moved R19 46.3 mm to (148.3, 76.0)
- moved C2 43.3 mm to (142.0, 84.4), turned to -90 degrees
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Connections:
- C1 pad 1: GND -> 12V
- C1 pad 2: -12V -> CV GND
- C2 pad 2: GND -> CV GND
- C3 pad 1: GND -> CV GND
- C3 pad 2: 5V -> -12V
- C4 pad 1: GND -> 12V
- C4 pad 2: 5V -> CV GND
- EURO_POWER1 pad 3: GND -> CV GND
- EURO_POWER1 pad 4: GND -> CV GND
- EURO_POWER1 pad 5: GND -> CV GND
- EURO_POWER1 pad 6: GND -> CV GND
- EURO_POWER1 pad 7: GND -> CV GND
- EURO_POWER1 pad 8: GND -> CV GND
- J2 pad 1: GND -> i2c SCL
- J2 pad 10: Out A LED Return Backboard -> Net-(J2-Pin_10)
- J2 pad 2: GND -> CV GND
- J2 pad 3: Out H LED Return Backboard -> i2c SDA
- J2 pad 4: Out G LED Return Backboard -> CV GND
- J2 pad 5: Out F LED Return Backboard -> i2c SCL
- J2 pad 6: Out E LED Return Backboard -> +5V from Host
- J2 pad 7: Out D LED Return Backboard -> i2c SDA
- J2 pad 8: Out C LED Return Backboard -> +5V from Host
- J2 pad 9: Out B LED Return Backboard -> Net-(J2-Pin_9)
- J3 pad 1: Out D LED Frontboard -> 3.3V
- J3 pad 2: Out C LED Frontboard -> Net-(J3-Pin_2)
- J4 pad 1: Out D LED Backboard -> 3.3V
- J4 pad 2: Out C LED Backboard -> Net-(J4-Pin_2)
- J5 pad 1: Out H LED Backboard -> 3.3v reference
- J5 pad 2: Out G LED Backboard -> 3.3v reference
- J5 pad 3: Out F LED Backboard -> DAC 1 Bias
- J5 pad 4: Out E LED Backboard -> DAC 3 Bias
- J5 pad 5: Output Backboard H -> 1.65v reference
- J5 pad 6: Output Backboard G -> 1.65v reference
- J5 pad 7: Output Backboard F -> 3.3v reference
- J5 pad 8: Output Backboard E -> 3.3v reference
- R1 pad 1: DAC output 2 -> 12V
- R1 pad 2: Net-(U3C-+) -> 5v reference
- R10 pad 1: GND -> Net-(U1B--)
- R10 pad 2: Out A LED Return Backboard -> Net-(C11-Pad2)
- R11 pad 1: DAC output 4 -> Net-(C10-Pad2)
- R11 pad 2: Net-(U5C-+) -> Net-(U1C-+)
- R12 pad 1: DAC output 3 -> Net-(C11-Pad2)
- R12 pad 2: Net-(U5A-+) -> Net-(U1D-+)
- R13 pad 1: Net-(R13-Pad1) -> CV GND
- R13 pad 2: Net-(U5C-+) -> Out A LED Return Backboard
- R14 pad 1: Net-(R14-Pad1) -> CV GND
- R14 pad 2: Net-(U5A-+) -> Out B LED Return Backboard
- R15 pad 1: GND -> Net-(U1C-+)
- R15 pad 2: Net-(U5C--) -> Output Backboard A
- R16 pad 1: GND -> Net-(U1D-+)
- R16 pad 2: Net-(U5A--) -> Output Backboard B
- R17 pad 1: Output Backboard D -> DAC output 3
- R17 pad 2: Net-(U5C--) -> Net-(U2A--)
- R18 pad 1: Output Backboard C -> DAC output 4
- R18 pad 2: Net-(U5A--) -> Net-(U2B--)
- R19 pad 1: GND -> Net-(U2A--)
- R19 pad 2: Out D LED Return Backboard -> Net-(C14-Pad2)
- R2 pad 1: DAC output 1 -> 12V
- R2 pad 2: Net-(U3A-+) -> 3.3v reference
- R20 pad 1: GND -> Net-(U2B--)
- R20 pad 2: Out C LED Return Backboard -> Net-(C15-Pad2)
- R21 pad 1: DAC output 6 -> Net-(C14-Pad2)
- R21 pad 2: Net-(U1C-+) -> Net-(U2C-+)
- R22 pad 1: DAC output 5 -> Net-(C15-Pad2)
- R22 pad 2: Net-(U1A-+) -> Net-(U2D-+)
- R23 pad 1: Net-(R23-Pad1) -> CV GND
- R23 pad 2: Net-(U1C-+) -> Out C LED Return Backboard
- R24 pad 1: Net-(R24-Pad1) -> CV GND
- R24 pad 2: Net-(U1A-+) -> Out D LED Return Backboard
- R25 pad 1: GND -> Net-(U2C-+)
- R25 pad 2: Net-(U1C--) -> Output Backboard C
- R26 pad 1: GND -> Net-(U2D-+)
- R26 pad 2: Net-(U1A--) -> Output Backboard D
- R3 pad 1: Net-(R3-Pad1) -> 3.3v reference
- R3 pad 2: Net-(U3C-+) -> 1.65v reference
- R4 pad 1: Net-(R4-Pad1) -> 1.65v reference
- R4 pad 2: Net-(U3A-+) -> CV GND
- R5 pad 1: GND -> Net-(J3-Pin_2)
- R5 pad 2: Net-(U3C--) -> i2c SDA
- R6 pad 1: GND -> Net-(J4-Pin_2)
- R6 pad 2: Net-(U3A--) -> i2c SCL
- R7 pad 1: Output Backboard B -> DAC output 1
- R7 pad 2: Net-(U3C--) -> Net-(U1A--)
- R8 pad 1: Output Backboard A -> DAC output 2
- R8 pad 2: Net-(U3A--) -> Net-(U1B--)
- R9 pad 1: GND -> Net-(U1A--)
- R9 pad 2: Out B LED Return Backboard -> Net-(C10-Pad2)
- U1 pad 1: Output Backboard E -> Net-(C10-Pad2)
- U1 pad 12: Output Backboard F -> Net-(U1D-+)
- U1 pad 13: Out F LED Return Backboard -> Out B LED Return Backboard
- U1 pad 14: Out F LED Backboard -> Out B LED Backboard
- U1 pad 3: Net-(U1A-+) -> DAC 1 Bias
- U1 pad 5: Output Backboard E -> DAC 2 Bias
- U1 pad 6: Out E LED Return Backboard -> Net-(U1B--)
- U1 pad 7: Out E LED Backboard -> Net-(C11-Pad2)
- U1 pad 8: Output Backboard F -> Out A LED Backboard
- U1 pad 9: Net-(U1C--) -> Out A LED Return Backboard
- U2 pad 1: Output Backboard G -> Net-(C14-Pad2)
- U2 pad 12: Output Backboard H -> Net-(U2D-+)
- U2 pad 13: Out H LED Return Backboard -> Out D LED Return Backboard
- U2 pad 14: Out H LED Backboard -> Out D LED Backboard
- U2 pad 3: Net-(U2A-+) -> DAC 3 Bias
- U2 pad 5: Output Backboard G -> DAC 4 Bias
- U2 pad 6: Out G LED Return Backboard -> Net-(U2B--)
- U2 pad 7: Out G LED Backboard -> Net-(C15-Pad2)
- U2 pad 8: Output Backboard H -> Out C LED Backboard
- U2 pad 9: Net-(U2C--) -> Out C LED Return Backboard
- U3 pad 1: Output Backboard A -> 5v reference
- U3 pad 2: Net-(U3A--) -> CV GND
- U3 pad 3: Net-(U3A-+) -> unconnected-(U3-NC-Pad3)
- U4 pad 1: 5V -> CV GND
- U4 pad 2: i2c SDA -> 3.3V
- U4 pad 3: i2c SCL -> 5V
- U4 pad 4: unconnected-(U4-~{LDAC}-Pad4) -> (no net)
- U5 pad 1: Output Backboard C -> 3.3v reference
- U5 pad 2: Net-(U5A--) -> CV GND
- U5 pad 3: Net-(U5A-+) -> unconnected-(U5-NC-Pad3)
Routing:
- net CV GND: track 0.00 -> 298.7 mm, vias 0 -> 24
- net 5V: track 0.00 -> 176.9 mm, vias 0 -> 3
- net GND: track 162.7 -> 0.00 mm, vias 15 -> 0
- net i2c SDA: track 0.00 -> 127.8 mm, vias 0 -> 1
- net i2c SCL: track 0.00 -> 125.8 mm, vias 0 -> 1
- net Output Frontboard B: track 123.6 -> 0.00 mm
- net 3.3V: track 0.00 -> 110.4 mm, vias 0 -> 1
- net Output Frontboard A: track 107.9 -> 0.00 mm
- net Normal C: track 0.00 -> 104.7 mm
- net 3.3v reference: track 0.00 -> 99.3 mm, vias 0 -> 2
- net Output Frontboard H: track 98.0 -> 0.00 mm
- net Out G LED Return Frontboard: track 90.9 -> 0.00 mm, vias 1 -> 0
- net Normal A: track 0.00 -> 85.8 mm, vias 0 -> 1
- net Net-(U5A-+): track 85.1 -> 0.00 mm, vias 2 -> 0
- net Output Frontboard G: track 84.8 -> 0.00 mm
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- added copper zone on B.Cu, net CV GND
- added copper zone on F.Cu, net CV GND
- removed copper zone on F.Cu, net GND
Other:
- board size 112.5 x 128.5 mm -> 86.1 x 128.5 mm
- board text added: "(c) doctea Tyrell Corporation"
- board text added: "1"
- board text added: "2"
- board text added: "4"
- board text added: "5v"
- board text added: "5v+3v3"
- board text added: "8"
- board text added: "A"
- board text added: "B"
- board text added: "C"
- board text added: "CV in"
- board text added: "CV out"
- board text added: "D"
- board text added: "JLCJLCJLCJLC"
- board text added: "bi"
- board text added: "dac1+3"
- board text added: "dac2+4"
- board text added: "gnd"
- board text added: "i2c expander"
- board text added: "redredredred"
- board text added: "uni"

Commit message: fixed incorrectly reversed analog input pins *facepalm*
Connections:
- ASD1015_2_ANA1 pad 2: Input Frontboard C -> Input Frontboard A
- ASD1015_2_ANA1 pad 4: Input Frontboard A -> Input Frontboard C
Routing:
- net Input Frontboard C: track 31.9 -> 18.3 mm
- net Input Frontboard A: track 10.2 -> 6.12 mm
- net CV GND: track 298.7 -> 297.8 mm
- net 5V: track 176.9 -> 176.3 mm
Changed lines of the file:
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@@
 			(layers "*.Cu" "*.Mask")
 			(remove_unused_layers no)
-			(net 56 "Input Frontboard C")
+			(net 55 "Input Frontboard A")
 			(pinfunction "Pin_2")
 			(pintype "passive")
@@
 			(layers "*.Cu" "*.Mask")
 			(remove_unused_layers no)
-			(net 55 "Input Frontboard A")
+			(net 56 "Input Frontboard C")
 			(pinfunction "Pin_4")
 			(pintype "passive")
@@
 	)
 	(segment
-		(start 152.2003 83.3323)
-		(end 151.926 83.058)
-		(width 0.25)
-		(layer "F.Cu")
-		(net 1)
-	)
-	(segment
 		(start 153.416 45.1612)
 		(end 153.416 44.3699)
@@
 		(net 1)
 	)
-	(segment
-		(start 149.4696 83.058)
-		(end 149.4571 83.0705)
-		(width 0.25)
-		(layer "F.Cu")
-		(net 1)
-	)
 	(via
 		(at 153.416 45.1612)
@@
 	)
 	(segment
-		(start 149.9108 101.4554)
-		(end 149.9108 101.5746)
-		(width 0.25)
-		(layer "F.Cu")
-		(net 3)
-	)
-	(segment
 		(start 143.503404 61.2446)
 		(end 141.9222 62.825804)
@@
 	)
 	(segment
-		(start 143.7136 95.3122)
-		(end 143.4224 95.3122)
-		(width 0.25)
-		(layer "F.Cu")
-		(net 3)
-	)
-	(segment
 		(start 137.5372 88.9681)
 		(end 137.5372 71.628)
@@
 	)
 	(segment
-		(start 161.3362 83.3882)
-		(end 161.484 83.536)
-		(width 0.25)
-		(layer "B.Cu")
-		(net 3)
-	)
-	(segment
 		(start 130.8354 102.87)
 		(end 130.8354 107.020901)
@@
 	)
 	(segment
-		(start 131.669499 106.879099)
-		(end 131.669499 106.6358)
-		(width 0.25)
-		(layer "B.Cu")
-		(net 5)
-	)
-	(segment
 		(start 136.2456 83.1596)
 		(end 138.2014 81.2038)
@@
 	)
 	(segment
-		(start 136.0926 88.3926)
-		(end 136.2456 88.2396)
-		(width 0.25)
-		(layer "B.Cu")
-		(net 5)
-	)
-	(segment
 		(start 149.7584 128.3716)
 		(end 149.7584 121.1072)
@@
 	(segment
 		(start 147.2516 25.1714)
-		(end 148.4246 26.3444)
+		(end 148.8772 26.797)
 		(width 0.25)
 		(layer "B.Cu")
@@
 	)
 	(segment
-		(start 148.8772 26.797)
-		(end 148.4246 26.3444)
-		(width 0.25)
-		(layer "B.Cu")
-		(net 18)
-	)
-	(segment
 		(start 151.257 26.797)
 		(end 148.8772 26.797)
@@
 	)
 	(segment
-		(start 142.8684 110.9726)
-		(end 142.8684 111.229096)
-		(width 0.25)
-		(layer "F.Cu")
-		(net 20)
-	)
-	(segment
 		(start 135.1534 48.927749)
 		(end 139.6204 53.394749)
@@
 		(net 20)
 	)
-	(segment
-		(start 142.9912 105.2562)
-		(end 142.7836 105.2562)
-		(width 0.25)
-		(layer "F.Cu")
-		(net 20)
-	)
 	(via
 		(at 134.8232 109.2708)
@@
 	)
 	(segment
-		(start 145.2514 39.6165)
-		(end 145.2514 39.7523)
-		(width 0.25)
-		(layer "F.Cu")
-		(net 21)
-	)
-	(segment
 		(start 150.0714 36.576)
 		(end 148.2919 36.576)
@@
 	)
 	(segment
-		(start 143.4244 92.9148)
-		(end 143.4416 92.932)
-		(width 0.25)
-		(layer "F.Cu")
-		(net 25)
-	)
-	(segment
 		(start 143.4244 90.9066)
 		(end 143.4244 92.9148)
@@
 	)
 	(segment
-		(start 145.4244 90.9066)
-		(end 145.8374 90.9066)
-		(width 0.25)
-		(layer "F.Cu")
-		(net 26)
-	)
-	(segment
 		(start 153.279695 78.9178)
 		(end 150.396995 81.8005)
@@
 	)
 	(segment
-		(start 136.819196 102.3148)
-		(end 136.5172 102.012804)
-		(width 0.25)
-		(layer "F.Cu")
-		(net 32)
-	)
-	(segment
 		(start 169.6532 43.1104)
 		(end 169.672 43.1292)
@@
 	)
 	(segment
-		(start 143.7136 99.9122)
-		(end 144.004 99.9122)
-		(width 0.25)
-		(layer "F.Cu")
-		(net 32)
-	)
-	(segment
 		(start 146.1614 62.5446)
 		(end 147.1676 63.5508)
@@
 	)
 	(segment
-		(start 164.0632 95.0214)
-		(end 163.9362 94.8944)
-		(width 0.25)
-		(layer "B.Cu")
-		(net 32)
-	)
-	(segment
 		(start 141.4272 92.9132)
 		(end 141.1732 92.6592)
@@
 	)
 	(segment
-		(start 144.637 104.8832)
-		(end 144.6276 104.8926)
-		(width 0.25)
-		(layer "F.Cu")
-		(net 45)
-	)
-	(segment
 		(start 137.558948 64.033297)
 		(end 137.558948 67.0254)
@@
 	)
 	(segment
-		(start 149.9108 108.6866)
-		(end 154.7466 103.8508)
-		(width 0.25)
-		(layer "B.Cu")
-		(net 55)
-	)
-	(segment
-		(start 149.9108 109.1946)
-		(end 149.9108 108.6866)
+		(start 149.9108 104.1146)
+		(end 151.6402 104.1146)
 		(width 0.25)
-		(layer "B.Cu")
+		(layer "F.Cu")
 		(net 55)
 	)
 	(segment
-		(start 154.7466 103.8508)
+		(start 151.6402 104.1146)
 		(end 154.7466 101.0082)
 		(width 0.25)
-		(layer "B.Cu")
-		(net 55)
-	)
-	(segment
-		(start 153.924 104.1146)
-		(end 154.7368 104.9274)
-		(width 0.25)
 		(layer "F.Cu")
-		(net 56)
+		(net 55)
 	)
 	(segment
-		(start 160.147 120.0578)
+		(start 153.6716 124.3832)
 		(end 154.7466 125.4582)
 		(width 0.25)
@@
 	)
 	(segment
-		(start 154.7368 104.9274)
-		(end 157.7594 104.9274)
+		(start 153.6716 112.9554)
+		(end 153.6716 124.3832)
 		(width 0.25)
 		(layer "F.Cu")
@@
 	)
 	(segment
-		(start 157.7594 104.9274)
-		(end 160.147 107.315)
-		(width 0.25)
-		(layer "F.Cu")
-		(net 56)
-	)
-	(segment
-		(start 160.147 107.315)
-		(end 160.147 120.0578)
-		(width 0.25)
-		(layer "F.Cu")
-		(net 56)
-	)
-	(segment
-		(start 149.9108 104.1146)
-		(end 153.924 104.1146)
+		(start 149.9108 109.1946)
+		(end 153.6716 112.9554)
 		(width 0.25)
 		(layer "F.Cu")
@@
 		(width 0.25)
 		(layer "F.Cu")
-		(net 64)
-	)
-	(segment
-		(start 145.5166 92.932)
-		(end 145.5166 92.6189)
-		(width 0.25)
-		(layer "F.Cu")

Commit message: removed some redundant traces
Connections:
- ASD1015_2_ANA1 pad 2: Input Frontboard A -> Input Frontboard C
- ASD1015_2_ANA1 pad 4: Input Frontboard C -> Input Frontboard A
Routing:
- net Input Frontboard C: track 18.3 -> 31.9 mm
- net CV GND: track 297.8 -> 285.2 mm
- net Input Frontboard A: track 6.12 -> 10.2 mm
- net 5V: track 176.3 -> 176.9 mm
- net DAC output 1: track 29.4 -> 30.0 mm
